Commit message: Rename packages and repo references from soarm to so_arm
Renamed soarm_description -> so_arm_description and soarm_control ->
so_arm_control (directories, package.xml names, CMakeLists project()
names, xacro find()/package:// references, launch FindPackageShare
calls, and controller names in the ros2_control yaml configs) to
match the GitHub remote rename from soarm_ros2 to so_arm_ros2.

Co-Authored-By: Claude Sonnet 5 <noreply@anthropic.com>

File: so_arm_description/urdf/so100/so100.urdf.xacro (robot description, xacro)
@@ -1,6 +1,6 @@
 <?xml version="1.0"?>
 <robot name="so100" xmlns:xacro="http://www.ros.org/wiki/xacro">
-  <xacro:include filename="$(find soarm_description)/urdf/so100/so100.common.xacro"/>
-  <xacro:include filename="$(find soarm_description)/urdf/so100/so100.control.xacro"/>
+  <xacro:include filename="$(find so_arm_description)/urdf/so100/so100.common.xacro"/>
+  <xacro:include filename="$(find so_arm_description)/urdf/so100/so100.control.xacro"/>
   <!-- Arguments (externally settable, default to property values in so100.control.xacro) -->
   <xacro:arg name="serial_port"    default="${serial_port}"/>
@@ -31,5 +31,5 @@
       <origin xyz="0 0 0" rpy="0 0 ${base_offset_rz}"/>
       <geometry>
-        <mesh filename="package://soarm_description/meshes/so100/Base.stl"/>
+        <mesh filename="package://so_arm_description/meshes/so100/Base.stl"/>
       </geometry>
       <material name="light_grey"/>
@@ -38,5 +38,5 @@
       <origin xyz="0 0 0" rpy="0 0 ${base_offset_rz}"/>
       <geometry>
-        <mesh filename="package://soarm_description/meshes/so100/Base_Motor.stl"/>
+        <mesh filename="package://so_arm_description/meshes/so100/Base_Motor.stl"/>
       </geometry>
       <material name="charcoal"/>
@@ -45,5 +45,5 @@
       <origin xyz="0 0 0" rpy="0 0 ${base_offset_rz}"/>
       <geometry>
-        <mesh filename="package://soarm_description/meshes/so100/Base.stl"/>
+        <mesh filename="package://so_arm_description/meshes/so100/Base.stl"/>
       </geometry>
     </collision>
@@ -59,5 +59,5 @@
       <origin xyz="0 0 0" rpy="${shoulder_offset_rx} 0 ${shoulder_offset_rz}"/>
       <geometry>
-        <mesh filename="package://soarm_description/meshes/so100/Rotation_Pitch.stl"/>
+        <mesh filename="package://so_arm_description/meshes/so100/Rotation_Pitch.stl"/>
       </geometry>
       <material name="light_grey"/>
@@ -66,5 +66,5 @@
       <origin xyz="0 0 0" rpy="${shoulder_offset_rx} 0 ${shoulder_offset_rz}"/>
       <geometry>
-        <mesh filename="package://soarm_description/meshes/so100/Rotation_Pitch_Motor.stl"/>
+        <mesh filename="package://so_arm_description/meshes/so100/Rotation_Pitch_Motor.stl"/>
       </geometry>
       <material name="charcoal"/>
@@ -73,5 +73,5 @@
       <origin xyz="0 0 0" rpy="${shoulder_offset_rx} 0 ${shoulder_offset_rz}"/>
       <geometry>
-        <mesh filename="package://soarm_description/meshes/so100/Rotation_Pitch.stl"/>
+        <mesh filename="package://so_arm_description/meshes/so100/Rotation_Pitch.stl"/>
       </geometry>
     </collision>
@@ -87,5 +87,5 @@
       <origin xyz="0 0 0" rpy="0 ${upper_arm_visual_ry} 0"/>
       <geometry>
-        <mesh filename="package://soarm_description/meshes/so100/Upper_Arm.stl"/>
+        <mesh filename="package://so_arm_description/meshes/so100/Upper_Arm.stl"/>
       </geometry>
       <material name="light_grey"/>
@@ -94,5 +94,5 @@
       <origin xyz="0 0 0" rpy="0 ${upper_arm_visual_ry} 0"/>
       <geometry>
-        <mesh filename="package://soarm_description/meshes/so100/Upper_Arm_Motor.stl"/>
+        <mesh filename="package://so_arm_description/meshes/so100/Upper_Arm_Motor.stl"/>
       </geometry>
       <material name="charcoal"/>
@@ -101,5 +101,5 @@
       <origin xyz="0 0 0" rpy="0 ${upper_arm_visual_ry} 0"/>
       <geometry>
-        <mesh filename="package://soarm_description/meshes/so100/Upper_Arm.stl"/>
+        <mesh filename="package://so_arm_description/meshes/so100/Upper_Arm.stl"/>
       </geometry>
     </collision>
@@ -115,5 +115,5 @@
       <origin xyz="0 0 0" rpy="0 ${lower_arm_visual_ry} 0"/>
       <geometry>
-        <mesh filename="package://soarm_description/meshes/so100/Lower_Arm.stl"/>
+        <mesh filename="package://so_arm_description/meshes/so100/Lower_Arm.stl"/>
       </geometry>
       <material name="light_grey"/>
@@ -122,5 +122,5 @@
       <origin xyz="0 0 0" rpy="0 ${lower_arm_visual_ry} 0"/>
       <geometry>
-        <mesh filename="package://soarm_description/meshes/so100/Lower_Arm_Motor.stl"/>
+        <mesh filename="package://so_arm_description/meshes/so100/Lower_Arm_Motor.stl"/>
       </geometry>
       <material name="charcoal"/>
@@ -129,5 +129,5 @@
       <origin xyz="0 0 0" rpy="0 ${lower_arm_visual_ry} 0"/>
       <geometry>
-        <mesh filename="package://soarm_description/meshes/so100/Lower_Arm.stl"/>
+        <mesh filename="package://so_arm_description/meshes/so100/Lower_Arm.stl"/>
       </geometry>
     </collision>
@@ -143,5 +143,5 @@
       <origin xyz="0 0 0" rpy="0 ${wrist_visual_ry} 0"/>
       <geometry>
-        <mesh filename="package://soarm_description/meshes/so100/Wrist_Pitch_Roll.stl"/>
+        <mesh filename="package://so_arm_description/meshes/so100/Wrist_Pitch_Roll.stl"/>
       </geometry>
       <material name="light_grey"/>
@@ -150,5 +150,5 @@
       <origin xyz="0 0 0" rpy="0 ${wrist_visual_ry} 0"/>
       <geometry>
-        <mesh filename="package://soarm_description/meshes/so100/Wrist_Pitch_Roll_Motor.stl"/>
+        <mesh filename="package://so_arm_description/meshes/so100/Wrist_Pitch_Roll_Motor.stl"/>
       </geometry>
       <material name="charcoal"/>
@@ -157,5 +157,5 @@
       <origin xyz="0 0 0" rpy="0 ${wrist_visual_ry} 0"/>
       <geometry>
-        <mesh filename="package://soarm_description/meshes/so100/Wrist_Pitch_Roll.stl"/>
+        <mesh filename="package://so_arm_description/meshes/so100/Wrist_Pitch_Roll.stl"/>
       </geometry>
     </collision>
@@ -171,5 +171,5 @@
       <origin xyz="0 0 0" rpy="${gripper_visual_rx} 0 0"/>
       <geometry>
-        <mesh filename="package://soarm_description/meshes/so100/Fixed_Jaw.stl"/>
+        <mesh filename="package://so_arm_description/meshes/so100/Fixed_Jaw.stl"/>
       </geometry>
       <material name="light_grey"/>
@@ -178,5 +178,5 @@
       <origin xyz="0 0 0" rpy="${gripper_visual_rx} 0 0"/>
       <geometry>
-        <mesh filename="package://soarm_description/meshes/so100/Fixed_Jaw_Motor.stl"/>
+        <mesh filename="package://so_arm_description/meshes/so100/Fixed_Jaw_Motor.stl"/>
       </geometry>
       <material name="charcoal"/>
@@ -192,5 +192,5 @@
     <visual>
       <geometry>
-        <mesh filename="package://soarm_description/meshes/so100/Moving_Jaw.stl"/>
+        <mesh filename="package://so_arm_description/meshes/so100/Moving_Jaw.stl"/>
       </geometry>
       <material name="light_grey"/>

File: so_arm_description/urdf/so101/so101.urdf.xacro (robot description, xacro)
@@ -1,6 +1,6 @@
 <?xml version="1.0"?>
 <robot name="so101" xmlns:xacro="http://www.ros.org/wiki/xacro">
-  <xacro:include filename="$(find soarm_description)/urdf/so101/so101.common.xacro"/>
-  <xacro:include filename="$(find soarm_description)/urdf/so101/so101.control.xacro"/>
+  <xacro:include filename="$(find so_arm_description)/urdf/so101/so101.common.xacro"/>
+  <xacro:include filename="$(find so_arm_description)/urdf/so101/so101.control.xacro"/>
   <!-- Arguments (externally settable, default to property values in so101.control.xacro) -->
   <xacro:arg name="serial_port"    default="${serial_port}"/>
@@ -31,5 +31,5 @@
       <origin xyz="-0.00636471 -9.94414e-05 -0.0024" rpy="1.5708 -1.67685e-15 1.5708"/>
       <geometry>
-        <mesh filename="package://soarm_description/meshes/so101/base_motor_holder_so101_v1.stl"/>
+        <mesh filename="package://so_arm_description/meshes/so101/base_motor_holder_so101_v1.stl"/>
       </geometry>
       <material name="light_grey"/>
@@ -38,5 +38,5 @@
       <origin xyz="-0.00636471 -9.94414e-05 -0.0024" rpy="1.5708 -1.67685e-15 1.5708"/>
       <geometry>
-        <mesh filename="package://soarm_description/meshes/so101/base_motor_holder_so101_v1.stl"/>
+        <mesh filename="package://so_arm_description/meshes/so101/base_motor_holder_so101_v1.stl"/>
       </geometry>
     </collision>
@@ -44,5 +44,5 @@
       <origin xyz="-0.00636471 -8.97657e-09 -0.0024" rpy="1.5708 -2.78073e-29 1.5708"/>
       <geometry>
-        <mesh filename="package://soarm_description/meshes/so101/base_so101_v2.stl"/>
+        <mesh filename="package://so_arm_description/meshes/so101/base_so101_v2.stl"/>
       </geometry>
       <material name="light_grey"/>
@@ -51,5 +51,5 @@
       <origin xyz="-0.00636471 -8.97657e-09 -0.0024" rpy="1.5708 -2.78073e-29 1.5708"/>
       <geometry>
-        <mesh filename="package://soarm_description/meshes/so101/base_so101_v2.stl"/>
+        <mesh filename="package://so_arm_description/meshes/so101/base_so101_v2.stl"/>
       </geometry>
     </collision>
@@ -57,5 +57,5 @@
       <origin xyz="0.0263353 -8.97657e-09 0.0437" rpy="-8.21148e-16 7.84513e-18 1.249e-15"/>
       <geometry>
-        <mesh filename="package://soarm_description/meshes/so101/sts3215_03a_v1.stl"/>
+        <mesh filename="package://so_arm_description/meshes/so101/sts3215_03a_v1.stl"/>
       </geometry>
       <material name="charcoal"/>
@@ -64,5 +64,5 @@
       <origin xyz="0.0263353 -8.97657e-09 0.0437" rpy="-8.21148e-16 7.84513e-18 1.249e-15"/>
       <geometry>
-        <mesh filename="package://soarm_description/meshes/so101/sts3215_03a_v1.stl"/>
+        <mesh filename="package://so_arm_description/meshes/so101/sts3215_03a_v1.stl"/>
       </geometry>
     </collision>
@@ -70,5 +70,5 @@
       <origin xyz="-0.0309827 -0.000199441 0.0474" rpy="1.5708 -1.35493e-14 1.5708"/>
       <geometry>
-        <mesh filename="package://soarm_description/meshes/so101/waveshare_mounting_plate_so101_v2.stl"/>
+        <mesh filename="package://so_arm_description/meshes/so101/waveshare_mounting_plate_so101_v2.stl"/>
       </geometry>
       <material name="light_grey"/>
@@ -77,5 +77,5 @@
       <origin xyz="-0.0309827 -0.000199441 0.0474" rpy="1.5708 -1.35493e-14 1.5708"/>
       <geometry>
-        <mesh filename="package://soarm_description/meshes/so101/waveshare_mounting_plate_so101_v2.stl"/>
+        <mesh filename="package://so_arm_description/meshes/so101/waveshare_mounting_plate_so101_v2.stl"/>
       </geometry>
     </collision>
@@ -91,5 +91,5 @@
       <origin xyz="0.0303992 0.000422241 0.0417" rpy="1.5708 -1.5708 0"/>
       <geometry>
-        <mesh filename="package://soarm_description/meshes/so101/sts3215_03a_v1.stl"/>
+        <mesh filename="package://so_arm_description/meshes/so101/sts3215_03a_v1.stl"/>
       </geometry>
       <material name="charcoal"/>
@@ -98,5 +98,5 @@
       <origin xyz="0.0303992 0.000422241 0.0417" rpy="1.5708 -1.5708 0"/>
       <geometry>
-        <mesh filename="package://soarm_description/meshes/so101/sts3215_03a_v1.stl"/>
+        <mesh filename="package://so_arm_description/meshes/so101/sts3215_03a_v1.stl"/>
       </geometry>
     </collision>
@@ -104,5 +104,5 @@
       <origin xyz="0.0675992 -0.000177759 -0.0158499" rpy="1.5708 1.5708 0"/>
       <geometry>
-        <mesh filename="package://soarm_description/meshes/so101/motor_holder_so101_base_v1.stl"/>
+        <mesh filename="package://so_arm_description/meshes/so101/motor_holder_so101_base_v1.stl"/>
       </geometry>
       <material name="light_grey"/>
@@ -111,5 +111,5 @@
       <origin xyz="0.0675992 -0.000177759 -0.0158499" rpy="1.5708 1.5708 0"/>
       <geometry>
-        <mesh filename="package://soarm_description/meshes/so101/motor_holder_so101_base_v1.stl"/>
+        <mesh filename="package://so_arm_description/meshes/so101/motor_holder_so101_base_v1.stl"/>
       </geometry>
     </collision>
@@ -117,5 +117,5 @@
       <origin xyz="-0.0122008 2.22413e-05 -0.0464" rpy="1.5708 0 3.14159"/>
       <geometry>
-        <mesh filename="package://soarm_description/meshes/so101/rotation_pitch_so101_v1.stl"/>
+        <mesh filename="package://so_arm_description/meshes/so101/rotation_pitch_so101_v1.stl"/>
       </geometry>
       <material name="light_grey"/>
@@ -124,5 +124,5 @@
       <origin xyz="-0.0122008 2.22413e-05 -0.0464" rpy="1.5708 0 3.14159"/>
       <geometry>
-        <mesh filename="package://soarm_description/meshes/so101/rotation_pitch_so101_v1.stl"/>
+        <mesh filename="package://so_arm_description/meshes/so101/rotation_pitch_so101_v1.stl"/>
       </geometry>
     </collision>
@@ -138,5 +138,5 @@
       <origin xyz="-0.11257 -0.0155 0.0187" rpy="-3.14159 -5.27356e-16 -1.5708"/>
       <geometry>
-        <mesh filename="package://soarm_description/meshes/so101/sts3215_03a_v1.stl"/>
+        <mesh filename="package://so_arm_description/meshes/so101/sts3215_03a_v1.stl"/>
       </geometry>
       <material name="charcoal"/>
@@ -145,5 +145,5 @@
       <origin xyz="-0.11257 -0.0155 0.0187" rpy="-3.14159 -5.27356e-16 -1.5708"/>
       <geometry>
-        <mesh filename="package://soarm_description/meshes/so101/sts3215_03a_v1.stl"/>
+        <mesh filename="package://so_arm_description/meshes/so101/sts3215_03a_v1.stl"/>
       </geometry>
     </collision>
@@ -151,5 +151,5 @@
       <origin xyz="-0.065085 0.012 0.0182" rpy="3.14159 -0 -1.30911e-30"/>
       <geometry>
-        <mesh filename="package://soarm_description/meshes/so101/upper_arm_so101_v1.stl"/>
+        <mesh filename="package://so_arm_description/meshes/so101/upper_arm_so101_v1.stl"/>
       </geometry>
       <material name="light_grey"/>
@@ -158,5 +158,5 @@
       <origin xyz="-0.065085 0.012 0.0182" rpy="3.14159 -0 -1.30911e-30"/>
       <geometry>
-        <mesh filename="package://soarm_description/meshes/so101/upper_arm_so101_v1.stl"/>
+        <mesh filename="package://so_arm_description/meshes/so101/upper_arm_so101_v1.stl"/>
       </geometry>
     </collision>
@@ -172,5 +172,5 @@
       <origin xyz="-0.0648499 -0.032 0.0182" rpy="3.14159 -0 6.67202e-31"/>
       <geometry>
-        <mesh filename="package://soarm_description/meshes/so101/under_arm_so101_v1.stl"/>
+        <mesh filename="package://so_arm_description/meshes/so101/under_arm_so101_v1.stl"/>
       </geometry>
       <material name="light_grey"/>
@@ -179,5 +179,5 @@
       <origin xyz="-0.0648499 -0.032 0.0182" rpy="3.14159 -0 6.67202e-31"/>
       <geometry>
-        <mesh filename="package://soarm_description/meshes/so101/under_arm_so101_v1.stl"/>
+        <mesh filename="package://so_arm_description/meshes/so101/under_arm_so101_v1.stl"/>
       </geometry>
     </collision>
@@ -185,5 +185,5 @@
       <origin xyz="-0.0648499 -0.032 0.018" rpy="-3.14159 -2.55351e-15 -1.83387e-30"/>
       <geometry>
-        <mesh filename="package://soarm_description/meshes/so101/motor_holder_so101_wrist_v1.stl"/>
+        <mesh filename="package://so_arm_description/meshes/so101/motor_holder_so101_wrist_v1.stl"/>
       </geometry>
       <material name="light_grey"/>
@@ -192,5 +192,5 @@
       <origin xyz="-0.0648499 -0.032 0.018" rpy="-3.14159 -2.55351e-15 -1.83387e-30"/>
       <geometry>
-        <mesh filename="package://soarm_description/meshes/so101/motor_holder_so101_wrist_v1.stl"/>
+        <mesh filename="package://so_arm_description/meshes/so101/motor_holder_so101_wrist_v1.stl"/>
       </geometry>
     </collision>
@@ -198,5 +198,5 @@
       <origin xyz="-0.1224 0.0052 0.0187" rpy="-3.14159 -7.88861e-31 -3.14159"/>
       <geometry>
-        <mesh filename="package://soarm_description/meshes/so101/sts3215_03a_v1.stl"/>
+        <mesh filename="package://so_arm_description/meshes/so101/sts3215_03a_v1.stl"/>
       </geometry>
       <material name="charcoal"/>
@@ -205,5 +205,5 @@
       <origin xyz="-0.1224 0.0052 0.0187" rpy="-3.14159 -7.88861e-31 -3.14159"/>
       <geometry>
-        <mesh filename="package://soarm_description/meshes/so101/sts3215_03a_v1.stl"/>
+        <mesh filename="package://so_arm_description/meshes/so101/sts3215_03a_v1.stl"/>
       </geometry>
     </collision>
@@ -219,5 +219,5 @@
       <origin xyz="8.32667e-17 -0.0424 0.0306" rpy="1.5708 1.5708 0"/>
       <geometry>
-        <mesh filename="package://soarm_description/meshes/so101/sts3215_03a_no_horn_v1.stl"/>
+        <mesh filename="package://so_arm_description/meshes/so101/sts3215_03a_no_horn_v1.stl"/>
       </geometry>
       <material name="charcoal"/>
@@ -226,5 +226,5 @@
       <origin xyz="8.32667e-17 -0.0424 0.0306" rpy="1.5708 1.5708 0"/>
       <geometry>
-        <mesh filename="package://soarm_description/meshes/so101/sts3215_03a_no_horn_v1.stl"/>
+        <mesh filename="package://so_arm_description/meshes/so101/sts3215_03a_no_horn_v1.stl"/>
       </geometry>
     </collision>
@@ -232,5 +232,5 @@
       <origin xyz="0 -0.028 0.0181" rpy="-1.5708 -1.5708 0"/>
       <geometry>
-        <mesh filename="package://soarm_description/meshes/so101/wrist_roll_pitch_so101_v2.stl"/>
+        <mesh filename="package://so_arm_description/meshes/so101/wrist_roll_pitch_so101_v2.stl"/>
       </geometry>
       <material name="light_grey"/>
@@ -239,5 +239,5 @@
       <origin xyz="0 -0.028 0.0181" rpy="-1.5708 -1.5708 0"/>
       <geometry>
-        <mesh filename="package://soarm_description/meshes/so101/wrist_roll_pitch_so101_v2.stl"/>
+        <mesh filename="package://so_arm_description/meshes/so101/wrist_roll_pitch_so101_v2.stl"/>
       </geometry>
     </collision>
@@ -253,5 +253,5 @@
       <origin xyz="0.0077 0.0001 -0.0234" rpy="-1.5708 -5.19179e-17 -1.66533e-16"/>
       <geometry>
-        <mesh filename="package://soarm_description/meshes/so101/sts3215_03a_v1.stl"/>
+        <mesh filename="package://so_arm_description/meshes/so101/sts3215_03a_v1.stl"/>
       </geometry>
       <material name="charcoal"/>
@@ -260,5 +260,5 @@
       <origin xyz="0.0077 0.0001 -0.0234" rpy="-1.5708 -5.19179e-17 -1.66533e-16"/>
       <geometry>
-        <mesh filename="package://soarm_description/meshes/so101/sts3215_03a_v1.stl"/>
+        <mesh filename="package://so_arm_description/meshes/so101/sts3215_03a_v1.stl"/>
       </geometry>
     </collision>
@@ -266,5 +266,5 @@
       <origin xyz="8.32667e-17 -0.000218214 0.000949706" rpy="-3.14159 -5.55112e-17 0"/>
       <geometry>
-        <mesh filename="package://soarm_description/meshes/so101/wrist_roll_follower_so101_v1.stl"/>
+        <mesh filename="package://so_arm_description/meshes/so101/wrist_roll_follower_so101_v1.stl"/>
       </geometry>
       <material name="light_grey"/>
@@ -273,5 +273,5 @@
       <origin xyz="8.32667e-17 -0.000218214 0.000949706" rpy="-3.14159 -5.55112e-17 0"/>
       <geometry>
-        <mesh filename="package://soarm_description/meshes/so101/wrist_roll_follower_so101_v1.stl"/>
+        <mesh filename="package://so_arm_description/meshes/so101/wrist_roll_follower_so101_v1.stl"/>
       </geometry>
     </collision>
@@ -295,5 +295,5 @@
       <origin xyz="-5.55112e-17 -5.55112e-17 0.0189" rpy="9.53145e-17 6.93889e-18 1.24077e-24"/>
       <geometry>
-        <mesh filename="package://soarm_description/meshes/so101/moving_jaw_so101_v1.stl"/>
+        <mesh filename="package://so_arm_description/meshes/so101/moving_jaw_so101_v1.stl"/>
       </geometry>
       <material name="light_grey"/>
@@ -302,5 +302,5 @@
       <origin xyz="-5.55112e-17 -5.55112e-17 0.0189" rpy="9.53145e-17 6.93889e-18 1.24077e-24"/>
       <geometry>
-        <mesh filename="package://soarm_description/meshes/so101/moving_jaw_so101_v1.stl"/>
+        <mesh filename="package://so_arm_description/meshes/so101/moving_jaw_so101_v1.stl"/>
       </geometry>
     </collision>
