Commit message: Add so_arm_control node stack, teleop/waypoint patrol, and README
Rebuilds so_arm_control as an ament_python package (replacing the earlier
ament_cmake skeleton): Pinocchio-based Cartesian IK joystick teleop
(ik_teleop_node), a self-collision-checked JointState->JointTrajectory
bridge (joint_trajectory_bridge_node), gripper teleop with velocity/
acceleration-matched motion (gripper_teleop_node), a priority-ordered
N-way joint command switch (joint_state_switch_node), a generic SetBool
toggle wrapper (bool_toggle_node), and lekiwi-style waypoint recording/
patrolling with per-waypoint gripper state and dwell time
(waypoint_recorder_node). Shared IK/kinematic-limiting and self-collision
checking code lives under so_arm_control/so_arm_utils/.

Also: control.launch.py/teleop.launch.py, config for both so100/so101,
generate_srdf.py, so_arm_description MJCF support, sts_hardware_interface
as a submodule under dependencies/ (not yet initialized - run
`git submodule update --init` after cloning), and a top-level README.

Co-Authored-By: Claude Sonnet 5 <noreply@anthropic.com>

File: so_arm_description/urdf/so100/so100.common.xacro (robot description, xacro)
@@ -26,3 +26,7 @@
   <xacro:property name="gripper_xyz" value="-0.0202 0 -0.0244"/>
   <xacro:property name="gripper_rpy" value="${pi/2} 0 ${pi}"/>
+  <!-- Estimated from Fixed_Jaw.stl's bbox (no onshape calibration for so100, unlike so101) -
+       reach axis/depth are mesh-verified, but rpy's left/up assignment is unverified (no photo). -->
+  <xacro:property name="end_effector_xyz" value="0.0025 0.0 -0.106"/>
+  <xacro:property name="end_effector_rpy" value="0 ${pi/2} 0"/>
 </robot>

File: so_arm_description/urdf/so100/so100.control.xacro (robot description, xacro)
@@ -17,5 +17,6 @@
   <xacro:property name="sts_max_velocity_steps" value="3400"/>  <!-- Max hardware velocity in steps/s -->
   <!-- Maximum allowable torque/velocity for each motor -->
-  <xacro:property name="max_velocity_rads" value="${sts_max_velocity_steps*2*pi/4096}"/>  <!-- rad/s -->
+  <xacro:property name="max_velocity_steps" value="${int(sts_max_velocity_steps * 0.85)}"/>  <!-- 85% of hardware max, 15% safety margin -->
+  <xacro:property name="max_velocity_rads" value="${max_velocity_steps*2*pi/4096}"/>  <!-- rad/s -->
   <xacro:property name="max_torque_nm" value="2.942"/>  <!-- N⋅m (30 kgf⋅cm for STS3215) -->
   <!-- Joint limits -->

File: so_arm_description/urdf/so100/so100.urdf (robot description, URDF)
Before this commit: robot so100, 8 links, 7 joints
Links:
- removed link jaw_link
- added link end_effector_link, mass 1e-9
- added link moving_jaw_link, mass 0.0202444; collision mesh filename=../../meshes/so100/Moving_Jaw.stl; visual mesh filename=../../meshes/so100/Moving_Jaw.stl
- link base_link: geometry collision mesh filename=../../meshes/so100/Base.stl; collision mesh filename=../../meshes/so100/Base_Motor.stl
- link gripper_link: geometry collision mesh filename=../../meshes/so100/Fixed_Jaw.stl; collision mesh filename=../../meshes/so100/Fixed_Jaw_Motor.stl
- link lower_arm_link: geometry collision mesh filename=../../meshes/so100/Lower_Arm.stl; collision mesh filename=../../meshes/so100/Lower_Arm_Motor.stl
- link shoulder_link: geometry collision mesh filename=../../meshes/so100/Rotation_Pitch.stl; collision mesh filename=../../meshes/so100/Rotation_Pitch_Motor.stl
- link upper_arm_link: geometry collision mesh filename=../../meshes/so100/Upper_Arm.stl; collision mesh filename=../../meshes/so100/Upper_Arm_Motor.stl
- link wrist_link: geometry collision mesh filename=../../meshes/so100/Wrist_Pitch_Roll.stl; collision mesh filename=../../meshes/so100/Wrist_Pitch_Roll_Motor.stl
Joints:
- removed joint base_footprint_joint
- added joint end_effector_joint: type fixed, parent gripper_link, child end_effector_link, origin xyz=0.0025 0.0 -0.106 rpy=0 1.5707963267948966 0
- added joint world_to_base: type fixed, parent base_footprint, child base_link, origin xyz=0 0 0 rpy=0 0 0
- joint elbow_flex_joint: limit lower=-3.14158 upper=0 effort=2.942 velocity=5.21553467881118 -> lower=-3.14158 upper=0 effort=2.942 velocity=1e6; origin xyz=-0.028 0.11257 0 rpy=0 0 1.5707963268 -> xyz=-0.028 0.11257 0 rpy=0 0 1.5707963267948966
- joint gripper_joint: child jaw_link -> moving_jaw_link; limit lower=-0.2 upper=2.0 effort=2.942 velocity=5.21553467881118 -> lower=-0.2 upper=2.0 effort=2.942 velocity=1e6; origin xyz=-0.0202 0 -0.0244 rpy=1.5707963268 0 3.1415926536 -> xyz=-0.0202 0 -0.0244 rpy=1.5707963267948966 0 3.141592653589793
- joint shoulder_lift_joint: limit lower=0 upper=3.5 effort=2.942 velocity=5.21553467881118 -> lower=0 upper=3.5 effort=2.942 velocity=1e6; origin xyz=0.0306 0 0.1025 rpy=-1.5707963268 1.3415926536 0 -> xyz=0.0306 0 0.1025 rpy=-1.5707963267948966 1.341592653589793 0
- joint shoulder_pan_joint: limit lower=-2 upper=2 effort=2.942 velocity=5.21553467881118 -> lower=-2 upper=2 effort=2.942 velocity=1e6
- joint wrist_flex_joint: limit lower=-2.5 upper=1.2 effort=2.942 velocity=5.21553467881118 -> lower=-2.5 upper=1.2 effort=2.942 velocity=1e6
- joint wrist_roll_joint: limit lower=-3.14158 upper=3.14158 effort=2.942 velocity=5.21553467881118 -> lower=-3.14158 upper=3.14158 effort=2.942 velocity=1e6; origin xyz=0 -0.0601 0 rpy=-1.5707963268 0 0 -> xyz=0 -0.0601 0 rpy=-1.5707963267948966 0 0

File: so_arm_description/urdf/so100/so100.urdf.xacro (robot description, xacro)
@@ -7,4 +7,14 @@
   <xacro:arg name="use_mock"       default="${use_mock}"/>
   <xacro:arg name="use_sync_write" default="${use_sync_write}"/>
+  <!-- Simulation backend selection.
+       "real" (default) uses the STS3215 serial hardware plugin below unchanged.
+       "mujoco" swaps the <hardware> plugin for mujoco_ros2_control/MujocoSystemInterface,
+       hosting the MJCF built from mjcf/so_arm.mjcf.xacro (so_arm_config:=so100) - see
+       so_arm_control/launch/control.launch.py. -->
+  <xacro:arg name="ros2_control_hardware_type" default="real"/>
+  <!-- mujoco mode only: path to the xacro-generated MJCF scene, and whether to open the
+       MuJoCo Simulate viewer window. -->
+  <xacro:arg name="mujoco_model" default=""/>
+  <xacro:arg name="mujoco_headless" default="false"/>
   <material name="light_grey">
     <color rgba="${light_grey_rgba}"/>
@@ -48,4 +58,10 @@
       </geometry>
     </collision>
+    <collision>
+      <origin xyz="0 0 0" rpy="0 0 ${base_offset_rz}"/>
+      <geometry>
+        <mesh filename="package://so_arm_description/meshes/so100/Base_Motor.stl"/>
+      </geometry>
+    </collision>
   </link>
   <!-- Shoulder link -->
@@ -76,4 +92,10 @@
       </geometry>
     </collision>
+    <collision>
+      <origin xyz="0 0 0" rpy="${shoulder_offset_rx} 0 ${shoulder_offset_rz}"/>
+      <geometry>
+        <mesh filename="package://so_arm_description/meshes/so100/Rotation_Pitch_Motor.stl"/>
+      </geometry>
+    </collision>
   </link>
   <!-- Upper arm link -->
@@ -104,4 +126,10 @@
       </geometry>
     </collision>
+    <collision>
+      <origin xyz="0 0 0" rpy="0 ${upper_arm_visual_ry} 0"/>
+      <geometry>
+        <mesh filename="package://so_arm_description/meshes/so100/Upper_Arm_Motor.stl"/>
+      </geometry>
+    </collision>
   </link>
   <!-- Lower arm link -->
@@ -132,4 +160,10 @@
       </geometry>
     </collision>
+    <collision>
+      <origin xyz="0 0 0" rpy="0 ${lower_arm_visual_ry} 0"/>
+      <geometry>
+        <mesh filename="package://so_arm_description/meshes/so100/Lower_Arm_Motor.stl"/>
+      </geometry>
+    </collision>
   </link>
   <!-- Wrist link -->
@@ -160,4 +194,10 @@
       </geometry>
     </collision>
+    <collision>
+      <origin xyz="0 0 0" rpy="0 ${wrist_visual_ry} 0"/>
+      <geometry>
+        <mesh filename="package://so_arm_description/meshes/so100/Wrist_Pitch_Roll_Motor.stl"/>
+      </geometry>
+    </collision>
   </link>
   <!-- Gripper link (fixed jaw) -->
@@ -175,14 +215,34 @@
       <material name="light_grey"/>
     </visual>
-    <visual>
+    <collision>
       <origin xyz="0 0 0" rpy="${gripper_visual_rx} 0 0"/>
       <geometry>
+        <mesh filename="package://so_arm_description/meshes/so100/Fixed_Jaw.stl"/>
+      </geometry>
+    </collision>
+    <visual>
+      <origin xyz="0 0 0" rpy="${gripper_visual_rx} 0 0"/>
+      <geometry>
         <mesh filename="package://so_arm_description/meshes/so100/Fixed_Jaw_Motor.stl"/>
       </geometry>
       <material name="charcoal"/>
     </visual>
+    <collision>
+      <origin xyz="0 0 0" rpy="${gripper_visual_rx} 0 0"/>
+      <geometry>
+        <mesh filename="package://so_arm_description/meshes/so100/Fixed_Jaw_Motor.stl"/>
+      </geometry>
+    </collision>
+  </link>
+  <!-- End effector frame (dummy link) -->
+  <link name="end_effector_link">
+    <inertial>
+      <origin xyz="0 0 0" rpy="0 0 0"/>
+      <mass value="1e-9"/>
+      <inertia ixx="0" ixy="0" ixz="0" iyy="0" iyz="0" izz="0"/>
+    </inertial>
   </link>
   <!-- Moving jaw link -->
-  <link name="jaw_link">
+  <link name="moving_jaw_link">
     <inertial>
       <mass value="0.0202444"/>
@@ -196,6 +256,13 @@
       <material name="light_grey"/>
     </visual>
+    <collision>
+      <geometry>
+        <mesh filename="package://so_arm_description/meshes/so100/Moving_Jaw.stl"/>
+      </geometry>
+    </collision>
   </link>
   <!-- JOINTS -->
+  <!-- velocity="1e6" (unreachable) disables JointSaturationLimiter's clipping - the real
+       ceiling comes from max_velocity in the <ros2_control> block below. -->
   <joint name="shoulder_pan_joint" type="revolute">
     <parent link="base_link"/>
@@ -203,5 +270,5 @@
     <origin xyz="${shoulder_pan_xyz}"/>
     <axis xyz="0 0 1"/>
-    <limit lower="${shoulder_pan_lower}" upper="${shoulder_pan_upper}" effort="${max_torque_nm}" velocity="${max_velocity_rads}"/>
+    <limit lower="${shoulder_pan_lower}" upper="${shoulder_pan_upper}" effort="${max_torque_nm}" velocity="1e6"/>
   </joint>
   <joint name="shoulder_lift_joint" type="revolute">
@@ -210,5 +277,5 @@
     <origin xyz="${shoulder_lift_xyz}" rpy="${shoulder_lift_rpy}"/>
     <axis xyz="0 0 1"/>
-    <limit lower="${shoulder_lift_lower}" upper="${shoulder_lift_upper}" effort="${max_torque_nm}" velocity="${max_velocity_rads}"/>
+    <limit lower="${shoulder_lift_lower}" upper="${shoulder_lift_upper}" effort="${max_torque_nm}" velocity="1e6"/>
   </joint>
   <joint name="elbow_flex_joint" type="revolute">
@@ -217,5 +284,5 @@
     <origin xyz="${elbow_flex_xyz}" rpy="${elbow_flex_rpy}"/>
     <axis xyz="0 0 1"/>
-    <limit lower="${elbow_flex_lower}" upper="${elbow_flex_upper}" effort="${max_torque_nm}" velocity="${max_velocity_rads}"/>
+    <limit lower="${elbow_flex_lower}" upper="${elbow_flex_upper}" effort="${max_torque_nm}" velocity="1e6"/>
   </joint>
   <joint name="wrist_flex_joint" type="revolute">
@@ -224,5 +291,5 @@
     <origin xyz="${wrist_flex_xyz}" rpy="${wrist_flex_rpy}"/>
     <axis xyz="0 0 1"/>
-    <limit lower="${wrist_flex_lower}" upper="${wrist_flex_upper}" effort="${max_torque_nm}" velocity="${max_velocity_rads}"/>
+    <limit lower="${wrist_flex_lower}" upper="${wrist_flex_upper}" effort="${max_torque_nm}" velocity="1e6"/>
   </joint>
   <joint name="wrist_roll_joint" type="revolute">
@@ -231,24 +298,36 @@
     <origin xyz="${wrist_roll_xyz}" rpy="${wrist_roll_rpy}"/>
     <axis xyz="0 0 1"/>
-    <limit lower="${wrist_roll_lower}" upper="${wrist_roll_upper}" effort="${max_torque_nm}" velocity="${max_velocity_rads}"/>
+    <limit lower="${wrist_roll_lower}" upper="${wrist_roll_upper}" effort="${max_torque_nm}" velocity="1e6"/>
   </joint>
   <joint name="gripper_joint" type="revolute">
     <parent link="gripper_link"/>
-    <child link="jaw_link"/>
+    <child link="moving_jaw_link"/>
     <origin xyz="${gripper_xyz}" rpy="${gripper_rpy}"/>
     <axis xyz="0 0 1"/>
-    <limit lower="${gripper_lower}" upper="${gripper_upper}" effort="${max_torque_nm}" velocity="${max_velocity_rads}"/>
+    <limit lower="${gripper_lower}" upper="${gripper_upper}" effort="${max_torque_nm}" velocity="1e6"/>
+  </joint>
+  <joint name="end_effector_joint" type="fixed">
+    <parent link="gripper_link"/>
+    <child link="end_effector_link"/>
+    <origin xyz="${end_effector_xyz}" rpy="${end_effector_rpy}"/>
   </joint>
   <!-- ROS 2 CONTROL -->
   <ros2_control name="so100_control" type="system">
     <hardware>
-      <plugin>sts_hardware_interface/STSHardwareInterface</plugin>
-      <param name="serial_port">$(arg serial_port)</param>
-      <param name="baud_rate">${baud_rate}</param>
-      <param name="communication_timeout_ms">100</param>
-      <param name="use_sync_write">$(arg use_sync_write)</param>
-      <param name="enable_mock_mode">$(arg use_mock)</param>
-      <param name="max_velocity_steps">${sts_max_velocity_steps}</param>
-      <param name="reset_states_on_activate">true</param>
+      <xacro:if value="${'$(arg ros2_control_hardware_type)' == 'mujoco'}">
+        <plugin>mujoco_ros2_control/MujocoSystemInterface</plugin>
+        <param name="mujoco_model">$(arg mujoco_model)</param>
+        <param name="headless">$(arg mujoco_headless)</param>
+      </xacro:if>
+      <xacro:if value="${'$(arg ros2_control_hardware_type)' == 'real'}">
+        <plugin>sts_hardware_interface/STSHardwareInterface</plugin>
+        <param name="serial_port">$(arg serial_port)</param>
+        <param name="baud_rate">${baud_rate}</param>
+        <param name="communication_timeout_ms">100</param>
+        <param name="use_sync_write">$(arg use_sync_write)</param>
+        <param name="enable_mock_mode">$(arg use_mock)</param>
+        <param name="max_velocity_steps">${sts_max_velocity_steps}</param>
+        <param name="reset_states_on_activate">true</param>
+      </xacro:if>
     </hardware>
     <joint name="shoulder_pan_joint">
@@ -260,11 +339,16 @@
       <param name="position_center_steps">2048</param>
       <command_interface name="position"/>
-      <state_interface name="position"/>
-      <state_interface name="velocity"/>
-      <state_interface name="effort"/>
-      <state_interface name="voltage"/>
-      <state_interface name="temperature"/>
-      <state_interface name="current"/>
-      <state_interface name="is_moving"/>
+      <command_interface name="velocity"/>
+      <state_interface name="position"/>
+      <state_interface name="velocity"/>
+      <state_interface name="effort"/>
+      <!-- Real-hardware-only telemetry: mujoco_ros2_control/MujocoSystemInterface doesn't
+           know these custom interface names. -->
+      <xacro:if value="${'$(arg ros2_control_hardware_type)' == 'real'}">
+        <state_interface name="voltage"/>
+        <state_interface name="temperature"/>
+        <state_interface name="current"/>
+        <state_interface name="is_moving"/>
+      </xacro:if>
     </joint>
     <joint name="shoulder_lift_joint">
@@ -276,11 +360,16 @@
       <param name="position_center_steps">2048</param>
       <command_interface name="position"/>
-      <state_interface name="position"/>
-      <state_interface name="velocity"/>
-      <state_interface name="effort"/>
-      <state_interface name="voltage"/>
-      <state_interface name="temperature"/>
-      <state_interface name="current"/>
-      <state_interface name="is_moving"/>
+      <command_interface name="velocity"/>
+      <state_interface name="position"/>
+      <state_interface name="velocity"/>
+      <state_interface name="effort"/>
+      <!-- Real-hardware-only telemetry: mujoco_ros2_control/MujocoSystemInterface doesn't
+           know these custom interface names. -->
+      <xacro:if value="${'$(arg ros2_control_hardware_type)' == 'real'}">
+        <state_interface name="voltage"/>
+        <state_interface name="temperature"/>
+        <state_interface name="current"/>
+        <state_interface name="is_moving"/>
+      </xacro:if>
     </joint>
     <joint name="elbow_flex_joint">
@@ -292,11 +381,16 @@
       <param name="position_center_steps">2048</param>
       <command_interface name="position"/>
-      <state_interface name="position"/>
-      <state_interface name="velocity"/>
-      <state_interface name="effort"/>
-      <state_interface name="voltage"/>
-      <state_interface name="temperature"/>
-      <state_interface name="current"/>
-      <state_interface name="is_moving"/>
+      <command_interface name="velocity"/>
+      <state_interface name="position"/>
+      <state_interface name="velocity"/>
+      <state_interface name="effort"/>
+      <!-- Real-hardware-only telemetry: mujoco_ros2_control/MujocoSystemInterface doesn't
+           know these custom interface names. -->
+      <xacro:if value="${'$(arg ros2_control_hardware_type)' == 'real'}">
+        <state_interface name="voltage"/>
+        <state_interface name="temperature"/>
+        <state_interface name="current"/>
+        <state_interface name="is_moving"/>
+      </xacro:if>
     </joint>
     <joint name="wrist_flex_joint">
@@ -308,11 +402,16 @@
       <param name="position_center_steps">2048</param>
       <command_interface name="position"/>
-      <state_interface name="position"/>
-      <state_interface name="velocity"/>
-      <state_interface name="effort"/>
-      <state_interface name="voltage"/>
-      <state_interface name="temperature"/>
-      <state_interface name="current"/>
-      <state_interface name="is_moving"/>
+      <command_interface name="velocity"/>
+      <state_interface name="position"/>
+      <state_interface name="velocity"/>
+      <state_interface name="effort"/>
+      <!-- Real-hardware-only telemetry: mujoco_ros2_control/MujocoSystemInterface doesn't
+           know these custom interface names. -->
+      <xacro:if value="${'$(arg ros2_control_hardware_type)' == 'real'}">
+        <state_interface name="voltage"/>
+        <state_interface name="temperature"/>
+        <state_interface name="current"/>
+        <state_interface name="is_moving"/>
+      </xacro:if>
     </joint>
     <joint name="wrist_roll_joint">
@@ -324,11 +423,16 @@
       <param name="position_center_steps">2048</param>
       <command_interface name="position"/>
-      <state_interface name="position"/>
-      <state_interface name="velocity"/>
-      <state_interface name="effort"/>
-      <state_interface name="voltage"/>
-      <state_interface name="temperature"/>
-      <state_interface name="current"/>
-      <state_interface name="is_moving"/>
+      <command_interface name="velocity"/>
+      <state_interface name="position"/>
+      <state_interface name="velocity"/>
+      <state_interface name="effort"/>
+      <!-- Real-hardware-only telemetry: mujoco_ros2_control/MujocoSystemInterface doesn't
+           know these custom interface names. -->
+      <xacro:if value="${'$(arg ros2_control_hardware_type)' == 'real'}">
+        <state_interface name="voltage"/>
+        <state_interface name="temperature"/>
+        <state_interface name="current"/>
+        <state_interface name="is_moving"/>
+      </xacro:if>
     </joint>
     <joint name="gripper_joint">
@@ -340,11 +444,16 @@
       <param name="position_center_steps">2048</param>
       <command_interface name="position"/>
-      <state_interface name="position"/>
-      <state_interface name="velocity"/>
-      <state_interface name="effort"/>
-      <state_interface name="voltage"/>
-      <state_interface name="temperature"/>
-      <state_interface name="current"/>
-      <state_interface name="is_moving"/>
+      <command_interface name="velocity"/>
+      <state_interface name="position"/>
+      <state_interface name="velocity"/>
+      <state_interface name="effort"/>
+      <!-- Real-hardware-only telemetry: mujoco_ros2_control/MujocoSystemInterface doesn't
+           know these custom interface names. -->
+      <xacro:if value="${'$(arg ros2_control_hardware_type)' == 'real'}">
+        <state_interface name="voltage"/>
+        <state_interface name="temperature"/>
+        <state_interface name="current"/>
+        <state_interface name="is_moving"/>
+      </xacro:if>
     </joint>
   </ros2_control>

File: so_arm_description/urdf/so101/so101.common.xacro (robot description, xacro)
@@ -16,5 +16,7 @@
   <xacro:property name="gripper_xyz" value="0.0202 0.0188 -0.0234"/>
   <xacro:property name="gripper_rpy" value="1.5708 -5.24284e-08 -1.41553e-15"/>
-  <xacro:property name="gripper_frame_xyz" value="-0.0079 -0.000218121 -0.0981274"/>
-  <xacro:property name="gripper_frame_rpy" value="0 3.14159 0"/>
+  <!-- end_effector_link's rpy (pitch pi/2, not the raw onshape TCP frame) makes its axes X=forward
+       Y=left Z=up like ik_target, instead of the arbitrary CAD TCP orientation. -->
+  <xacro:property name="end_effector_xyz" value="-0.0079 -0.000218121 -0.0981274"/>
+  <xacro:property name="end_effector_rpy" value="0 1.5708 0"/>
 </robot>

File: so_arm_description/urdf/so101/so101.control.xacro (robot description, xacro)
@@ -17,5 +17,6 @@
   <xacro:property name="sts_max_velocity_steps" value="3400"/>  <!-- Max hardware velocity in steps/s -->
   <!-- Maximum allowable torque/velocity for each motor -->
-  <xacro:property name="max_velocity_rads" value="${sts_max_velocity_steps*2*pi/4096}"/>  <!-- rad/s -->
+  <xacro:property name="max_velocity_steps" value="${int(sts_max_velocity_steps * 0.85)}"/>  <!-- 85% of hardware max, 15% safety margin -->
+  <xacro:property name="max_velocity_rads" value="${max_velocity_steps*2*pi/4096}"/>  <!-- rad/s -->
   <xacro:property name="max_torque_nm" value="2.942"/>  <!-- N⋅m (30 kgf⋅cm for STS3215) -->
   <!-- Joint limits (from onshape-to-robot calibration) -->
