Commit message: Add so_arm_control node stack, teleop/waypoint patrol, and README
Rebuilds so_arm_control as an ament_python package (replacing the earlier
ament_cmake skeleton): Pinocchio-based Cartesian IK joystick teleop
(ik_teleop_node), a self-collision-checked JointState->JointTrajectory
bridge (joint_trajectory_bridge_node), gripper teleop with velocity/
acceleration-matched motion (gripper_teleop_node), a priority-ordered
N-way joint command switch (joint_state_switch_node), a generic SetBool
toggle wrapper (bool_toggle_node), and lekiwi-style waypoint recording/
patrolling with per-waypoint gripper state and dwell time
(waypoint_recorder_node). Shared IK/kinematic-limiting and self-collision
checking code lives under so_arm_control/so_arm_utils/.

Also: control.launch.py/teleop.launch.py, config for both so100/so101,
generate_srdf.py, so_arm_description MJCF support, sts_hardware_interface
as a submodule under dependencies/ (not yet initialized - run
`git submodule update --init` after cloning), and a top-level README.

Co-Authored-By: Claude Sonnet 5 <noreply@anthropic.com>

File: so_arm_description/urdf/so101/so101.urdf (robot description, URDF)
Before this commit: robot so101, 9 links, 8 joints
Links:
- removed link gripper_frame_link
- added link end_effector_link, mass 1e-9
Joints:
- removed joint base_footprint_joint
- removed joint elbow_flex
- removed joint gripper
- removed joint gripper_frame_joint
- removed joint shoulder_lift
- removed joint shoulder_pan
- removed joint wrist_flex
- removed joint wrist_roll
- added joint elbow_flex_joint: type revolute, parent upper_arm_link, child lower_arm_link, origin xyz=-0.11257 -0.028 1.73763e-16 rpy=-3.63608e-16 8.74301e-16 1.5708, axis 0 0 1, limit lower=-1.69 upper=1.69 effort=2.942 velocity=1e6
- added joint end_effector_joint: type fixed, parent gripper_link, child end_effector_link, origin xyz=-0.0079 -0.000218121 -0.0981274 rpy=0 1.5708 0
- added joint gripper_joint: type revolute, parent gripper_link, child moving_jaw_link, origin xyz=0.0202 0.0188 -0.0234 rpy=1.5708 -5.24284e-08 -1.41553e-15, axis 0 0 1, limit lower=-0.174533 upper=1.74533 effort=2.942 velocity=1e6
- added joint shoulder_lift_joint: type revolute, parent shoulder_link, child upper_arm_link, origin xyz=0.0303992 -0.0182778 0.0542 rpy=-1.5708 1.5708 0, axis 0 0 1, limit lower=-1.74533 upper=1.74533 effort=2.942 velocity=1e6
- added joint shoulder_pan_joint: type revolute, parent base_link, child shoulder_link, origin xyz=0.0388353 -8.97657e-09 0.0624, axis 0 0 1, limit lower=-1.91986 upper=1.91986 effort=2.942 velocity=1e6
- added joint world_to_base: type fixed, parent base_footprint, child base_link, origin xyz=0 0 0 rpy=0 0 0
- added joint wrist_flex_joint: type revolute, parent lower_arm_link, child wrist_link, origin xyz=-0.1349 0.0052 3.62355e-17 rpy=4.02456e-15 8.67362e-16 -1.5708, axis 0 0 1, limit lower=-1.65806 upper=1.65806 effort=2.942 velocity=1e6
- added joint wrist_roll_joint: type revolute, parent wrist_link, child gripper_link, origin xyz=5.55112e-17 -0.0611 0.0181 rpy=1.5708 0.0486795 3.14159, axis 0 0 1, limit lower=-2.74385 upper=2.84121 effort=2.942 velocity=1e6

File: so_arm_description/urdf/so101/so101.urdf.xacro (robot description, xacro)
@@ -7,4 +7,14 @@
   <xacro:arg name="use_mock"       default="${use_mock}"/>
   <xacro:arg name="use_sync_write" default="${use_sync_write}"/>
+  <!-- Simulation backend selection.
+       "real" (default) uses the STS3215 serial hardware plugin below unchanged.
+       "mujoco" swaps the <hardware> plugin for mujoco_ros2_control/MujocoSystemInterface,
+       hosting the MJCF built from mjcf/so_arm.mjcf.xacro (so_arm_config:=so101) - see
+       so_arm_control/launch/control.launch.py. -->
+  <xacro:arg name="ros2_control_hardware_type" default="real"/>
+  <!-- mujoco mode only: path to the xacro-generated MJCF scene, and whether to open the
+       MuJoCo Simulate viewer window. -->
+  <xacro:arg name="mujoco_model" default=""/>
+  <xacro:arg name="mujoco_headless" default="false"/>
   <material name="light_grey">
     <color rgba="${light_grey_rgba}"/>
@@ -277,6 +287,6 @@
     </collision>
   </link>
-  <!-- Gripper frame (dummy link) -->
-  <link name="gripper_frame_link">
+  <!-- End effector frame (dummy link) -->
+  <link name="end_effector_link">
     <inertial>
       <origin xyz="0 0 0" rpy="0 0 0"/>
@@ -307,4 +317,6 @@
   </link>
   <!-- JOINTS -->
+  <!-- velocity="1e6" (unreachable) disables JointSaturationLimiter's clipping - the real
+       ceiling comes from max_velocity in the <ros2_control> block below. -->
   <joint name="shoulder_pan_joint" type="revolute">
     <parent link="base_link"/>
@@ -312,5 +324,5 @@
     <origin xyz="${shoulder_pan_xyz}"/>
     <axis xyz="0 0 1"/>
-    <limit lower="${shoulder_pan_lower}" upper="${shoulder_pan_upper}" effort="${max_torque_nm}" velocity="${max_velocity_rads}"/>
+    <limit lower="${shoulder_pan_lower}" upper="${shoulder_pan_upper}" effort="${max_torque_nm}" velocity="1e6"/>
   </joint>
   <joint name="shoulder_lift_joint" type="revolute">
@@ -319,5 +331,5 @@
     <origin xyz="${shoulder_lift_xyz}" rpy="${shoulder_lift_rpy}"/>
     <axis xyz="0 0 1"/>
-    <limit lower="${shoulder_lift_lower}" upper="${shoulder_lift_upper}" effort="${max_torque_nm}" velocity="${max_velocity_rads}"/>
+    <limit lower="${shoulder_lift_lower}" upper="${shoulder_lift_upper}" effort="${max_torque_nm}" velocity="1e6"/>
   </joint>
   <joint name="elbow_flex_joint" type="revolute">
@@ -326,5 +338,5 @@
     <origin xyz="${elbow_flex_xyz}" rpy="${elbow_flex_rpy}"/>
     <axis xyz="0 0 1"/>
-    <limit lower="${elbow_flex_lower}" upper="${elbow_flex_upper}" effort="${max_torque_nm}" velocity="${max_velocity_rads}"/>
+    <limit lower="${elbow_flex_lower}" upper="${elbow_flex_upper}" effort="${max_torque_nm}" velocity="1e6"/>
   </joint>
   <joint name="wrist_flex_joint" type="revolute">
@@ -333,5 +345,5 @@
     <origin xyz="${wrist_flex_xyz}" rpy="${wrist_flex_rpy}"/>
     <axis xyz="0 0 1"/>
-    <limit lower="${wrist_flex_lower}" upper="${wrist_flex_upper}" effort="${max_torque_nm}" velocity="${max_velocity_rads}"/>
+    <limit lower="${wrist_flex_lower}" upper="${wrist_flex_upper}" effort="${max_torque_nm}" velocity="1e6"/>
   </joint>
   <joint name="wrist_roll_joint" type="revolute">
@@ -340,10 +352,10 @@
     <origin xyz="${wrist_roll_xyz}" rpy="${wrist_roll_rpy}"/>
     <axis xyz="0 0 1"/>
-    <limit lower="${wrist_roll_lower}" upper="${wrist_roll_upper}" effort="${max_torque_nm}" velocity="${max_velocity_rads}"/>
-  </joint>
-  <joint name="gripper_frame_joint" type="fixed">
+    <limit lower="${wrist_roll_lower}" upper="${wrist_roll_upper}" effort="${max_torque_nm}" velocity="1e6"/>
+  </joint>
+  <joint name="end_effector_joint" type="fixed">
     <parent link="gripper_link"/>
-    <child link="gripper_frame_link"/>
-    <origin xyz="${gripper_frame_xyz}" rpy="${gripper_frame_rpy}"/>
+    <child link="end_effector_link"/>
+    <origin xyz="${end_effector_xyz}" rpy="${end_effector_rpy}"/>
   </joint>
   <joint name="gripper_joint" type="revolute">
@@ -352,17 +364,24 @@
     <origin xyz="${gripper_xyz}" rpy="${gripper_rpy}"/>
     <axis xyz="0 0 1"/>
-    <limit lower="${gripper_lower}" upper="${gripper_upper}" effort="${max_torque_nm}" velocity="${max_velocity_rads}"/>
+    <limit lower="${gripper_lower}" upper="${gripper_upper}" effort="${max_torque_nm}" velocity="1e6"/>
   </joint>
   <!-- ROS 2 CONTROL -->
   <ros2_control name="so101_control" type="system">
     <hardware>
-      <plugin>sts_hardware_interface/STSHardwareInterface</plugin>
-      <param name="serial_port">$(arg serial_port)</param>
-      <param name="baud_rate">${baud_rate}</param>
-      <param name="communication_timeout_ms">100</param>
-      <param name="use_sync_write">$(arg use_sync_write)</param>
-      <param name="enable_mock_mode">$(arg use_mock)</param>
-      <param name="max_velocity_steps">${sts_max_velocity_steps}</param>
-      <param name="reset_states_on_activate">true</param>
+      <xacro:if value="${'$(arg ros2_control_hardware_type)' == 'mujoco'}">
+        <plugin>mujoco_ros2_control/MujocoSystemInterface</plugin>
+        <param name="mujoco_model">$(arg mujoco_model)</param>
+        <param name="headless">$(arg mujoco_headless)</param>
+      </xacro:if>
+      <xacro:if value="${'$(arg ros2_control_hardware_type)' == 'real'}">
+        <plugin>sts_hardware_interface/STSHardwareInterface</plugin>
+        <param name="serial_port">$(arg serial_port)</param>
+        <param name="baud_rate">${baud_rate}</param>
+        <param name="communication_timeout_ms">100</param>
+        <param name="use_sync_write">$(arg use_sync_write)</param>
+        <param name="enable_mock_mode">$(arg use_mock)</param>
+        <param name="max_velocity_steps">${sts_max_velocity_steps}</param>
+        <param name="reset_states_on_activate">true</param>
+      </xacro:if>
     </hardware>
     <joint name="shoulder_pan_joint">
@@ -374,11 +393,16 @@
       <param name="position_center_steps">2048</param>
       <command_interface name="position"/>
+      <command_interface name="velocity"/>
       <state_interface name="position"/>
       <state_interface name="velocity"/>
       <state_interface name="effort"/>
-      <state_interface name="voltage"/>
-      <state_interface name="temperature"/>
-      <state_interface name="current"/>
-      <state_interface name="is_moving"/>
+      <!-- Real-hardware-only telemetry: mujoco_ros2_control/MujocoSystemInterface doesn't
+           know these custom interface names. -->
+      <xacro:if value="${'$(arg ros2_control_hardware_type)' == 'real'}">
+        <state_interface name="voltage"/>
+        <state_interface name="temperature"/>
+        <state_interface name="current"/>
+        <state_interface name="is_moving"/>
+      </xacro:if>
     </joint>
     <joint name="shoulder_lift_joint">
@@ -390,11 +414,16 @@
       <param name="position_center_steps">2048</param>
       <command_interface name="position"/>
+      <command_interface name="velocity"/>
       <state_interface name="position"/>
       <state_interface name="velocity"/>
       <state_interface name="effort"/>
-      <state_interface name="voltage"/>
-      <state_interface name="temperature"/>
-      <state_interface name="current"/>
-      <state_interface name="is_moving"/>
+      <!-- Real-hardware-only telemetry: mujoco_ros2_control/MujocoSystemInterface doesn't
+           know these custom interface names. -->
+      <xacro:if value="${'$(arg ros2_control_hardware_type)' == 'real'}">
+        <state_interface name="voltage"/>
+        <state_interface name="temperature"/>
+        <state_interface name="current"/>
+        <state_interface name="is_moving"/>
+      </xacro:if>
     </joint>
     <joint name="elbow_flex_joint">
@@ -406,11 +435,16 @@
       <param name="position_center_steps">2048</param>
       <command_interface name="position"/>
+      <command_interface name="velocity"/>
       <state_interface name="position"/>
       <state_interface name="velocity"/>
       <state_interface name="effort"/>
-      <state_interface name="voltage"/>
-      <state_interface name="temperature"/>
-      <state_interface name="current"/>
-      <state_interface name="is_moving"/>
+      <!-- Real-hardware-only telemetry: mujoco_ros2_control/MujocoSystemInterface doesn't
+           know these custom interface names. -->
+      <xacro:if value="${'$(arg ros2_control_hardware_type)' == 'real'}">
+        <state_interface name="voltage"/>
+        <state_interface name="temperature"/>
+        <state_interface name="current"/>
+        <state_interface name="is_moving"/>
+      </xacro:if>
     </joint>
     <joint name="wrist_flex_joint">
@@ -422,11 +456,16 @@
       <param name="position_center_steps">2048</param>
       <command_interface name="position"/>
+      <command_interface name="velocity"/>
       <state_interface name="position"/>
       <state_interface name="velocity"/>
       <state_interface name="effort"/>
-      <state_interface name="voltage"/>
-      <state_interface name="temperature"/>
-      <state_interface name="current"/>
-      <state_interface name="is_moving"/>
+      <!-- Real-hardware-only telemetry: mujoco_ros2_control/MujocoSystemInterface doesn't
+           know these custom interface names. -->
+      <xacro:if value="${'$(arg ros2_control_hardware_type)' == 'real'}">
+        <state_interface name="voltage"/>
+        <state_interface name="temperature"/>
+        <state_interface name="current"/>
+        <state_interface name="is_moving"/>
+      </xacro:if>
     </joint>
     <joint name="wrist_roll_joint">
@@ -438,11 +477,16 @@
       <param name="position_center_steps">2048</param>
       <command_interface name="position"/>
+      <command_interface name="velocity"/>
       <state_interface name="position"/>
       <state_interface name="velocity"/>
       <state_interface name="effort"/>
-      <state_interface name="voltage"/>
-      <state_interface name="temperature"/>
-      <state_interface name="current"/>
-      <state_interface name="is_moving"/>
+      <!-- Real-hardware-only telemetry: mujoco_ros2_control/MujocoSystemInterface doesn't
+           know these custom interface names. -->
+      <xacro:if value="${'$(arg ros2_control_hardware_type)' == 'real'}">
+        <state_interface name="voltage"/>
+        <state_interface name="temperature"/>
+        <state_interface name="current"/>
+        <state_interface name="is_moving"/>
+      </xacro:if>
     </joint>
     <joint name="gripper_joint">
@@ -454,11 +498,16 @@
       <param name="position_center_steps">2048</param>
       <command_interface name="position"/>
+      <command_interface name="velocity"/>
       <state_interface name="position"/>
       <state_interface name="velocity"/>
       <state_interface name="effort"/>
-      <state_interface name="voltage"/>
-      <state_interface name="temperature"/>
-      <state_interface name="current"/>
-      <state_interface name="is_moving"/>
+      <!-- Real-hardware-only telemetry: mujoco_ros2_control/MujocoSystemInterface doesn't
+           know these custom interface names. -->
+      <xacro:if value="${'$(arg ros2_control_hardware_type)' == 'real'}">
+        <state_interface name="voltage"/>
+        <state_interface name="temperature"/>
+        <state_interface name="current"/>
+        <state_interface name="is_moving"/>
+      </xacro:if>
     </joint>
   </ros2_control>
