Commit message: feat: streaming JTC velocity, servo PID/deadband, teleop speed tuning
- joint_trajectory_bridge: stream a cruise velocity derived from
  target delta/dt instead of always zero, so consecutive trajectory
  points chain into continuous motion instead of braking every tick.
- Remove the 85%-of-max speed cap; use the servo protocol's full u16
  velocity ceiling (65535) instead of a conservative 3400 guess, and
  let servo firmware enforce the real limit.
- Add per-joint STS servo PID (p/d/i_coefficient) and deadband
  (CW_DEAD/CCW_DEAD) params, wired through so100/so101 xacros into
  sts_hardware_interface (bumped submodule - see its own log).
- gripper_teleop_node: fix inverted joystick-to-position mapping.
- kinematics.py: raise IK Gauss-Newton _STEP for faster convergence.
- teleop.yaml: retune publish_rate/max_acceleration/twist scales to
  match the above.

Co-Authored-By: Claude Sonnet 5 <noreply@anthropic.com>

File: so_arm_description/urdf/so100/so100.control.xacro (robot description, xacro)
@@ -16,9 +16,15 @@
   <xacro:property name="gripper_operating_mode" value="0"/> <!-- Gripper joint 6: 0=Position, 1=Velocity, 2=PWM/Effort -->
   <!-- Motor-specific parameter (STS3215 default) -->
-  <xacro:property name="sts_max_velocity_steps" value="3400"/>  <!-- Max hardware velocity in steps/s -->
+  <xacro:property name="sts_max_velocity_steps" value="65535"/>  <!-- protocol's own u16 ceiling - let servo firmware, not us, set the real cap -->
   <!-- Maximum allowable torque/velocity for each motor -->
-  <xacro:property name="max_velocity_steps" value="${int(sts_max_velocity_steps * 0.85)}"/>  <!-- 85% of hardware max, 15% safety margin -->
+  <xacro:property name="max_velocity_steps" value="${sts_max_velocity_steps}"/>  <!-- full hardware max -->
   <xacro:property name="max_velocity_rads" value="${max_velocity_steps*2*pi/4096}"/>  <!-- rad/s -->
   <xacro:property name="max_torque_nm" value="2.942"/>  <!-- N⋅m (30 kgf⋅cm for STS3215) -->
+  <!-- Position-mode (Mode 0) internal servo PID, written to EEPROM on activate -->
+  <xacro:property name="p_coefficient" value="14"/>
+  <xacro:property name="d_coefficient" value="24"/>
+  <xacro:property name="i_coefficient" value="0"/>
+  <!-- Position insensitive-area (CW_DEAD/CCW_DEAD, both set to this value) -->
+  <xacro:property name="deadband" value="2"/>
   <!-- Joint limits -->
   <xacro:property name="shoulder_pan_lower" value="-2"/>

File: so_arm_description/urdf/so100/so100.urdf.xacro (robot description, xacro)
@@ -335,4 +335,8 @@
       <param name="max_velocity">${max_velocity_rads}</param>
       <param name="position_center_steps">2048</param>
+      <param name="p_coefficient">${p_coefficient}</param>
+      <param name="d_coefficient">${d_coefficient}</param>
+      <param name="i_coefficient">${i_coefficient}</param>
+      <param name="deadband">${deadband}</param>
       <!-- cmd interfaces depend on arm_operating_mode -->
       <xacro:if value="${'$(arg arm_operating_mode)' == '2'}">
@@ -361,4 +365,8 @@
       <param name="max_velocity">${max_velocity_rads}</param>
       <param name="position_center_steps">2048</param>
+      <param name="p_coefficient">${p_coefficient}</param>
+      <param name="d_coefficient">${d_coefficient}</param>
+      <param name="i_coefficient">${i_coefficient}</param>
+      <param name="deadband">${deadband}</param>
       <!-- cmd interfaces depend on arm_operating_mode -->
       <xacro:if value="${'$(arg arm_operating_mode)' == '2'}">
@@ -387,4 +395,8 @@
       <param name="max_velocity">${max_velocity_rads}</param>
       <param name="position_center_steps">2048</param>
+      <param name="p_coefficient">${p_coefficient}</param>
+      <param name="d_coefficient">${d_coefficient}</param>
+      <param name="i_coefficient">${i_coefficient}</param>
+      <param name="deadband">${deadband}</param>
       <!-- cmd interfaces depend on arm_operating_mode -->
       <xacro:if value="${'$(arg arm_operating_mode)' == '2'}">
@@ -413,4 +425,8 @@
       <param name="max_velocity">${max_velocity_rads}</param>
       <param name="position_center_steps">2048</param>
+      <param name="p_coefficient">${p_coefficient}</param>
+      <param name="d_coefficient">${d_coefficient}</param>
+      <param name="i_coefficient">${i_coefficient}</param>
+      <param name="deadband">${deadband}</param>
       <!-- cmd interfaces depend on arm_operating_mode -->
       <xacro:if value="${'$(arg arm_operating_mode)' == '2'}">
@@ -439,4 +455,8 @@
       <param name="max_velocity">${max_velocity_rads}</param>
       <param name="position_center_steps">2048</param>
+      <param name="p_coefficient">${p_coefficient}</param>
+      <param name="d_coefficient">${d_coefficient}</param>
+      <param name="i_coefficient">${i_coefficient}</param>
+      <param name="deadband">${deadband}</param>
       <!-- cmd interfaces depend on arm_operating_mode -->
       <xacro:if value="${'$(arg arm_operating_mode)' == '2'}">
@@ -465,4 +485,8 @@
       <param name="max_velocity">${max_velocity_rads}</param>
       <param name="position_center_steps">2048</param>
+      <param name="p_coefficient">${p_coefficient}</param>
+      <param name="d_coefficient">${d_coefficient}</param>
+      <param name="i_coefficient">${i_coefficient}</param>
+      <param name="deadband">${deadband}</param>
       <!-- cmd interfaces depend on gripper_operating_mode -->
       <xacro:if value="${'$(arg gripper_operating_mode)' == '2'}">

File: so_arm_description/urdf/so101/so101.control.xacro (robot description, xacro)
@@ -16,9 +16,15 @@
   <xacro:property name="gripper_operating_mode" value="0"/> <!-- Gripper joint 6: 0=Position, 1=Velocity, 2=PWM/Effort -->
   <!-- Motor-specific parameter (STS3215 default) -->
-  <xacro:property name="sts_max_velocity_steps" value="3400"/>  <!-- Max hardware velocity in steps/s -->
+  <xacro:property name="sts_max_velocity_steps" value="65535"/>  <!-- protocol's own u16 ceiling - let servo firmware, not us, set the real cap -->
   <!-- Maximum allowable torque/velocity for each motor -->
-  <xacro:property name="max_velocity_steps" value="${int(sts_max_velocity_steps * 0.85)}"/>  <!-- 85% of hardware max, 15% safety margin -->
+  <xacro:property name="max_velocity_steps" value="${sts_max_velocity_steps}"/>  <!-- full hardware max -->
   <xacro:property name="max_velocity_rads" value="${max_velocity_steps*2*pi/4096}"/>  <!-- rad/s -->
   <xacro:property name="max_torque_nm" value="2.942"/>  <!-- N⋅m (30 kgf⋅cm for STS3215) -->
+  <!-- Position-mode (Mode 0) internal servo PID, written to EEPROM on activate -->
+  <xacro:property name="p_coefficient" value="14"/>
+  <xacro:property name="d_coefficient" value="24"/>
+  <xacro:property name="i_coefficient" value="0"/>
+  <!-- Position insensitive-area (CW_DEAD/CCW_DEAD, both set to this value) -->
+  <xacro:property name="deadband" value="2"/>
   <!-- Joint limits (from onshape-to-robot calibration) -->
   <xacro:property name="shoulder_pan_lower" value="-1.91986"/>

File: so_arm_description/urdf/so101/so101.urdf.xacro (robot description, xacro)
@@ -437,5 +437,5 @@
     <child link="moving_jaw_link"/>
     <origin xyz="${gripper_xyz}" rpy="${gripper_rpy}"/>
-    <axis xyz="0 0 1"/>
+    <axis xyz="0 0 -1"/>
     <limit lower="${gripper_lower}" upper="${gripper_upper}" effort="${max_torque_nm}" velocity="1e6"/>
   </joint>
@@ -466,4 +466,8 @@
       <param name="max_velocity">${max_velocity_rads}</param>
       <param name="position_center_steps">2048</param>
+      <param name="p_coefficient">${p_coefficient}</param>
+      <param name="d_coefficient">${d_coefficient}</param>
+      <param name="i_coefficient">${i_coefficient}</param>
+      <param name="deadband">${deadband}</param>
       <!-- cmd interfaces depend on arm_operating_mode -->
       <xacro:if value="${'$(arg arm_operating_mode)' == '2'}">
@@ -492,4 +496,8 @@
       <param name="max_velocity">${max_velocity_rads}</param>
       <param name="position_center_steps">2048</param>
+      <param name="p_coefficient">${p_coefficient}</param>
+      <param name="d_coefficient">${d_coefficient}</param>
+      <param name="i_coefficient">${i_coefficient}</param>
+      <param name="deadband">${deadband}</param>
       <!-- cmd interfaces depend on arm_operating_mode -->
       <xacro:if value="${'$(arg arm_operating_mode)' == '2'}">
@@ -518,4 +526,8 @@
       <param name="max_velocity">${max_velocity_rads}</param>
       <param name="position_center_steps">2048</param>
+      <param name="p_coefficient">${p_coefficient}</param>
+      <param name="d_coefficient">${d_coefficient}</param>
+      <param name="i_coefficient">${i_coefficient}</param>
+      <param name="deadband">${deadband}</param>
       <!-- cmd interfaces depend on arm_operating_mode -->
       <xacro:if value="${'$(arg arm_operating_mode)' == '2'}">
@@ -544,4 +556,8 @@
       <param name="max_velocity">${max_velocity_rads}</param>
       <param name="position_center_steps">2048</param>
+      <param name="p_coefficient">${p_coefficient}</param>
+      <param name="d_coefficient">${d_coefficient}</param>
+      <param name="i_coefficient">${i_coefficient}</param>
+      <param name="deadband">${deadband}</param>
       <!-- cmd interfaces depend on arm_operating_mode -->
       <xacro:if value="${'$(arg arm_operating_mode)' == '2'}">
@@ -570,4 +586,8 @@
       <param name="max_velocity">${max_velocity_rads}</param>
       <param name="position_center_steps">2048</param>
+      <param name="p_coefficient">${p_coefficient}</param>
+      <param name="d_coefficient">${d_coefficient}</param>
+      <param name="i_coefficient">${i_coefficient}</param>
+      <param name="deadband">${deadband}</param>
       <!-- cmd interfaces depend on arm_operating_mode -->
       <xacro:if value="${'$(arg arm_operating_mode)' == '2'}">
@@ -596,4 +616,8 @@
       <param name="max_velocity">${max_velocity_rads}</param>
       <param name="position_center_steps">2048</param>
+      <param name="p_coefficient">${p_coefficient}</param>
+      <param name="d_coefficient">${d_coefficient}</param>
+      <param name="i_coefficient">${i_coefficient}</param>
+      <param name="deadband">${deadband}</param>
       <!-- cmd interfaces depend on gripper_operating_mode -->
       <xacro:if value="${'$(arg gripper_operating_mode)' == '2'}">
