Commit message: feat: split operating_mode into arm_operating_mode + gripper_operating_mode
Allows the gripper motor (joint 6) to run in a different operating mode
from the five arm joints, without changing any default behaviour (all
joints still default to mode 0/Position).

Changes:
- so100.control.xacro, so101.control.xacro:
    Rename 'operating_mode' property to 'arm_operating_mode'; add
    'gripper_operating_mode' property (both default 0).

- so100.urdf.xacro, so101.urdf.xacro:
    Replace single 'operating_mode' xacro:arg with two args:
      arm_operating_mode     (joints 1-5, default 0)
      gripper_operating_mode (joint 6,    default 0)
    Arm joints use arm_operating_mode; gripper_joint uses
    gripper_operating_mode for its operating_mode param and
    command_interface xacro:if/unless blocks.

- control.launch.py:
    Expose arm_operating_mode and gripper_operating_mode as launch args
    (default '0'). Both are always forwarded to xacro.

- gravity_comp.launch.py:
    Pass arm_operating_mode:=2 gripper_operating_mode:=2 (same
    behaviour as the previous operating_mode:=2).

- control.yaml:
    Add a comment on gripper_controller noting that mode 2 requires
    switching to effort_controllers/JointGroupEffortController.

Usage:
  # All joints position (default - unchanged):
  ros2 launch so_arm_control control.launch.py

  # Gripper in PWM/effort mode, arm in position mode:
  ros2 launch so_arm_control control.launch.py gripper_operating_mode:=2

File: so_arm_description/urdf/so100/so100.control.xacro (robot description, xacro)
@@ -13,5 +13,6 @@
   <xacro:property name="wrist_roll_motor_id" value="5"/>
   <xacro:property name="gripper_motor_id" value="6"/>
-  <xacro:property name="operating_mode" value="0"/>  <!-- Position mode -->
+  <xacro:property name="arm_operating_mode" value="0"/>     <!-- Arm joints 1-5: 0=Position, 1=Velocity, 2=PWM/Effort -->
+  <xacro:property name="gripper_operating_mode" value="0"/> <!-- Gripper joint 6: 0=Position, 1=Velocity, 2=PWM/Effort -->
   <!-- Motor-specific parameter (STS3215 default) -->
   <xacro:property name="sts_max_velocity_steps" value="3400"/>  <!-- Max hardware velocity in steps/s -->

File: so_arm_description/urdf/so100/so100.urdf.xacro (robot description, xacro)
@@ -10,6 +10,7 @@
        Changing this changes which <command_interface> below is generated (position+velocity
        vs. effort), so it can't be switched live - it's baked into robot_description at
-       hardware-interface startup. gravity_comp.launch.py overrides this to 2. -->
-  <xacro:arg name="operating_mode" default="${operating_mode}"/>
+       hardware-interface startup. gravity_comp.launch.py overrides both to 2. -->
+  <xacro:arg name="arm_operating_mode"     default="${arm_operating_mode}"/>     <!-- Joints 1-5 (shoulder → wrist) -->
+  <xacro:arg name="gripper_operating_mode" default="${gripper_operating_mode}"/> <!-- Joint 6 (gripper) -->
   <!-- Simulation backend selection.
        "real" (default) uses the STS3215 serial hardware plugin below unchanged.
@@ -338,5 +339,5 @@
     <joint name="shoulder_pan_joint">
       <param name="motor_id">${shoulder_pan_motor_id}</param>
-      <param name="operating_mode">$(arg operating_mode)</param>
+      <param name="operating_mode">$(arg arm_operating_mode)</param>
       <param name="min_position">${shoulder_pan_lower}</param>
       <param name="max_position">${shoulder_pan_upper}</param>
@@ -344,9 +345,9 @@
       <param name="position_center_steps">2048</param>
       <!-- Mode 0/1: position+velocity; Mode 2 (PWM/Effort): effort only - see the
-           operating_mode arg's own comment above for why this can't be a runtime switch. -->
-      <xacro:if value="${'$(arg operating_mode)' == '2'}">
+           arm_operating_mode arg's own comment above for why this can't be a runtime switch. -->
+      <xacro:if value="${'$(arg arm_operating_mode)' == '2'}">
         <command_interface name="effort"/>
       </xacro:if>
-      <xacro:unless value="${'$(arg operating_mode)' == '2'}">
+      <xacro:unless value="${'$(arg arm_operating_mode)' == '2'}">
         <command_interface name="position"/>
         <command_interface name="velocity"/>
@@ -366,5 +367,5 @@
     <joint name="shoulder_lift_joint">
       <param name="motor_id">${shoulder_lift_motor_id}</param>
-      <param name="operating_mode">$(arg operating_mode)</param>
+      <param name="operating_mode">$(arg arm_operating_mode)</param>
       <param name="min_position">${shoulder_lift_lower}</param>
       <param name="max_position">${shoulder_lift_upper}</param>
@@ -372,9 +373,9 @@
       <param name="position_center_steps">2048</param>
       <!-- Mode 0/1: position+velocity; Mode 2 (PWM/Effort): effort only - see the
-           operating_mode arg's own comment above for why this can't be a runtime switch. -->
-      <xacro:if value="${'$(arg operating_mode)' == '2'}">
+           arm_operating_mode arg's own comment above for why this can't be a runtime switch. -->
+      <xacro:if value="${'$(arg arm_operating_mode)' == '2'}">
         <command_interface name="effort"/>
       </xacro:if>
-      <xacro:unless value="${'$(arg operating_mode)' == '2'}">
+      <xacro:unless value="${'$(arg arm_operating_mode)' == '2'}">
         <command_interface name="position"/>
         <command_interface name="velocity"/>
@@ -394,5 +395,5 @@
     <joint name="elbow_flex_joint">
       <param name="motor_id">${elbow_flex_motor_id}</param>
-      <param name="operating_mode">$(arg operating_mode)</param>
+      <param name="operating_mode">$(arg arm_operating_mode)</param>
       <param name="min_position">${elbow_flex_lower}</param>
       <param name="max_position">${elbow_flex_upper}</param>
@@ -400,9 +401,9 @@
       <param name="position_center_steps">2048</param>
       <!-- Mode 0/1: position+velocity; Mode 2 (PWM/Effort): effort only - see the
-           operating_mode arg's own comment above for why this can't be a runtime switch. -->
-      <xacro:if value="${'$(arg operating_mode)' == '2'}">
+           arm_operating_mode arg's own comment above for why this can't be a runtime switch. -->
+      <xacro:if value="${'$(arg arm_operating_mode)' == '2'}">
         <command_interface name="effort"/>
       </xacro:if>
-      <xacro:unless value="${'$(arg operating_mode)' == '2'}">
+      <xacro:unless value="${'$(arg arm_operating_mode)' == '2'}">
         <command_interface name="position"/>
         <command_interface name="velocity"/>
@@ -422,5 +423,5 @@
     <joint name="wrist_flex_joint">
       <param name="motor_id">${wrist_flex_motor_id}</param>
-      <param name="operating_mode">$(arg operating_mode)</param>
+      <param name="operating_mode">$(arg arm_operating_mode)</param>
       <param name="min_position">${wrist_flex_lower}</param>
       <param name="max_position">${wrist_flex_upper}</param>
@@ -428,9 +429,9 @@
       <param name="position_center_steps">2048</param>
       <!-- Mode 0/1: position+velocity; Mode 2 (PWM/Effort): effort only - see the
-           operating_mode arg's own comment above for why this can't be a runtime switch. -->
-      <xacro:if value="${'$(arg operating_mode)' == '2'}">
+           arm_operating_mode arg's own comment above for why this can't be a runtime switch. -->
+      <xacro:if value="${'$(arg arm_operating_mode)' == '2'}">
         <command_interface name="effort"/>
       </xacro:if>
-      <xacro:unless value="${'$(arg operating_mode)' == '2'}">
+      <xacro:unless value="${'$(arg arm_operating_mode)' == '2'}">
         <command_interface name="position"/>
         <command_interface name="velocity"/>
@@ -450,5 +451,5 @@
     <joint name="wrist_roll_joint">
       <param name="motor_id">${wrist_roll_motor_id}</param>
-      <param name="operating_mode">$(arg operating_mode)</param>
+      <param name="operating_mode">$(arg arm_operating_mode)</param>
       <param name="min_position">${wrist_roll_lower}</param>
       <param name="max_position">${wrist_roll_upper}</param>
@@ -456,9 +457,9 @@
       <param name="position_center_steps">2048</param>
       <!-- Mode 0/1: position+velocity; Mode 2 (PWM/Effort): effort only - see the
-           operating_mode arg's own comment above for why this can't be a runtime switch. -->
-      <xacro:if value="${'$(arg operating_mode)' == '2'}">
+           arm_operating_mode arg's own comment above for why this can't be a runtime switch. -->
+      <xacro:if value="${'$(arg arm_operating_mode)' == '2'}">
         <command_interface name="effort"/>
       </xacro:if>
-      <xacro:unless value="${'$(arg operating_mode)' == '2'}">
+      <xacro:unless value="${'$(arg arm_operating_mode)' == '2'}">
         <command_interface name="position"/>
         <command_interface name="velocity"/>
@@ -478,5 +479,5 @@
     <joint name="gripper_joint">
       <param name="motor_id">${gripper_motor_id}</param>
-      <param name="operating_mode">$(arg operating_mode)</param>
+      <param name="operating_mode">$(arg gripper_operating_mode)</param>
       <param name="min_position">${gripper_lower}</param>
       <param name="max_position">${gripper_upper}</param>
@@ -484,9 +485,11 @@
       <param name="position_center_steps">2048</param>
       <!-- Mode 0/1: position+velocity; Mode 2 (PWM/Effort): effort only - see the
-           operating_mode arg's own comment above for why this can't be a runtime switch. -->
-      <xacro:if value="${'$(arg operating_mode)' == '2'}">
+           gripper_operating_mode arg's own comment above for why this can't be a runtime switch.
+           Note: when gripper_operating_mode=2, switch gripper_controller to
+           effort_controllers/JointGroupEffortController in control.yaml. -->
+      <xacro:if value="${'$(arg gripper_operating_mode)' == '2'}">
         <command_interface name="effort"/>
       </xacro:if>
-      <xacro:unless value="${'$(arg operating_mode)' == '2'}">
+      <xacro:unless value="${'$(arg gripper_operating_mode)' == '2'}">
         <command_interface name="position"/>
         <command_interface name="velocity"/>

File: so_arm_description/urdf/so101/so101.control.xacro (robot description, xacro)
@@ -13,5 +13,6 @@
   <xacro:property name="wrist_roll_motor_id" value="5"/>
   <xacro:property name="gripper_motor_id" value="6"/>
-  <xacro:property name="operating_mode" value="0"/>  <!-- Position mode -->
+  <xacro:property name="arm_operating_mode" value="0"/>     <!-- Arm joints 1-5: 0=Position, 1=Velocity, 2=PWM/Effort -->
+  <xacro:property name="gripper_operating_mode" value="0"/> <!-- Gripper joint 6: 0=Position, 1=Velocity, 2=PWM/Effort -->
   <!-- Motor-specific parameter (STS3215 default) -->
   <xacro:property name="sts_max_velocity_steps" value="3400"/>  <!-- Max hardware velocity in steps/s -->

File: so_arm_description/urdf/so101/so101.urdf.xacro (robot description, xacro)
@@ -10,6 +10,7 @@
        Changing this changes which <command_interface> below is generated (position+velocity
        vs. effort), so it can't be switched live - it's baked into robot_description at
-       hardware-interface startup. gravity_comp.launch.py overrides this to 2. -->
-  <xacro:arg name="operating_mode" default="${operating_mode}"/>
+       hardware-interface startup. gravity_comp.launch.py overrides both to 2. -->
+  <xacro:arg name="arm_operating_mode"     default="${arm_operating_mode}"/>     <!-- Joints 1-5 (shoulder → wrist) -->
+  <xacro:arg name="gripper_operating_mode" default="${gripper_operating_mode}"/> <!-- Joint 6 (gripper) -->
   <!-- Simulation backend selection.
        "real" (default) uses the STS3215 serial hardware plugin below unchanged.
@@ -469,5 +470,5 @@
     <joint name="shoulder_pan_joint">
       <param name="motor_id">${shoulder_pan_motor_id}</param>
-      <param name="operating_mode">$(arg operating_mode)</param>
+      <param name="operating_mode">$(arg arm_operating_mode)</param>
       <param name="min_position">${shoulder_pan_lower}</param>
       <param name="max_position">${shoulder_pan_upper}</param>
@@ -475,9 +476,9 @@
       <param name="position_center_steps">2048</param>
       <!-- Mode 0/1: position+velocity; Mode 2 (PWM/Effort): effort only - see the
-           operating_mode arg's own comment above for why this can't be a runtime switch. -->
-      <xacro:if value="${'$(arg operating_mode)' == '2'}">
+           arm_operating_mode arg's own comment above for why this can't be a runtime switch. -->
+      <xacro:if value="${'$(arg arm_operating_mode)' == '2'}">
         <command_interface name="effort"/>
       </xacro:if>
-      <xacro:unless value="${'$(arg operating_mode)' == '2'}">
+      <xacro:unless value="${'$(arg arm_operating_mode)' == '2'}">
         <command_interface name="position"/>
         <command_interface name="velocity"/>
@@ -497,5 +498,5 @@
     <joint name="shoulder_lift_joint">
       <param name="motor_id">${shoulder_lift_motor_id}</param>
-      <param name="operating_mode">$(arg operating_mode)</param>
+      <param name="operating_mode">$(arg arm_operating_mode)</param>
       <param name="min_position">${shoulder_lift_lower}</param>
       <param name="max_position">${shoulder_lift_upper}</param>
@@ -503,9 +504,9 @@
       <param name="position_center_steps">2048</param>
       <!-- Mode 0/1: position+velocity; Mode 2 (PWM/Effort): effort only - see the
-           operating_mode arg's own comment above for why this can't be a runtime switch. -->
-      <xacro:if value="${'$(arg operating_mode)' == '2'}">
+           arm_operating_mode arg's own comment above for why this can't be a runtime switch. -->
+      <xacro:if value="${'$(arg arm_operating_mode)' == '2'}">
         <command_interface name="effort"/>
       </xacro:if>
-      <xacro:unless value="${'$(arg operating_mode)' == '2'}">
+      <xacro:unless value="${'$(arg arm_operating_mode)' == '2'}">
         <command_interface name="position"/>
         <command_interface name="velocity"/>
@@ -525,5 +526,5 @@
     <joint name="elbow_flex_joint">
       <param name="motor_id">${elbow_flex_motor_id}</param>
-      <param name="operating_mode">$(arg operating_mode)</param>
+      <param name="operating_mode">$(arg arm_operating_mode)</param>
       <param name="min_position">${elbow_flex_lower}</param>
       <param name="max_position">${elbow_flex_upper}</param>
@@ -531,9 +532,9 @@
       <param name="position_center_steps">2048</param>
       <!-- Mode 0/1: position+velocity; Mode 2 (PWM/Effort): effort only - see the
-           operating_mode arg's own comment above for why this can't be a runtime switch. -->
-      <xacro:if value="${'$(arg operating_mode)' == '2'}">
+           arm_operating_mode arg's own comment above for why this can't be a runtime switch. -->
+      <xacro:if value="${'$(arg arm_operating_mode)' == '2'}">
         <command_interface name="effort"/>
       </xacro:if>
-      <xacro:unless value="${'$(arg operating_mode)' == '2'}">
+      <xacro:unless value="${'$(arg arm_operating_mode)' == '2'}">
         <command_interface name="position"/>
         <command_interface name="velocity"/>
@@ -553,5 +554,5 @@
     <joint name="wrist_flex_joint">
       <param name="motor_id">${wrist_flex_motor_id}</param>
-      <param name="operating_mode">$(arg operating_mode)</param>
+      <param name="operating_mode">$(arg arm_operating_mode)</param>
       <param name="min_position">${wrist_flex_lower}</param>
       <param name="max_position">${wrist_flex_upper}</param>
@@ -559,9 +560,9 @@
       <param name="position_center_steps">2048</param>
       <!-- Mode 0/1: position+velocity; Mode 2 (PWM/Effort): effort only - see the
-           operating_mode arg's own comment above for why this can't be a runtime switch. -->
-      <xacro:if value="${'$(arg operating_mode)' == '2'}">
+           arm_operating_mode arg's own comment above for why this can't be a runtime switch. -->
+      <xacro:if value="${'$(arg arm_operating_mode)' == '2'}">
         <command_interface name="effort"/>
       </xacro:if>
-      <xacro:unless value="${'$(arg operating_mode)' == '2'}">
+      <xacro:unless value="${'$(arg arm_operating_mode)' == '2'}">
         <command_interface name="position"/>
         <command_interface name="velocity"/>
@@ -581,5 +582,5 @@
     <joint name="wrist_roll_joint">
       <param name="motor_id">${wrist_roll_motor_id}</param>
-      <param name="operating_mode">$(arg operating_mode)</param>
+      <param name="operating_mode">$(arg arm_operating_mode)</param>
       <param name="min_position">${wrist_roll_lower}</param>
       <param name="max_position">${wrist_roll_upper}</param>
@@ -587,9 +588,9 @@
       <param name="position_center_steps">2048</param>
       <!-- Mode 0/1: position+velocity; Mode 2 (PWM/Effort): effort only - see the
-           operating_mode arg's own comment above for why this can't be a runtime switch. -->
-      <xacro:if value="${'$(arg operating_mode)' == '2'}">
+           arm_operating_mode arg's own comment above for why this can't be a runtime switch. -->
+      <xacro:if value="${'$(arg arm_operating_mode)' == '2'}">
         <command_interface name="effort"/>
       </xacro:if>
-      <xacro:unless value="${'$(arg operating_mode)' == '2'}">
+      <xacro:unless value="${'$(arg arm_operating_mode)' == '2'}">
         <command_interface name="position"/>
         <command_interface name="velocity"/>
@@ -609,5 +610,5 @@
     <joint name="gripper_joint">
       <param name="motor_id">${gripper_motor_id}</param>
-      <param name="operating_mode">$(arg operating_mode)</param>
+      <param name="operating_mode">$(arg gripper_operating_mode)</param>
       <param name="min_position">${gripper_lower}</param>
       <param name="max_position">${gripper_upper}</param>
@@ -615,9 +616,11 @@
       <param name="position_center_steps">2048</param>
       <!-- Mode 0/1: position+velocity; Mode 2 (PWM/Effort): effort only - see the
-           operating_mode arg's own comment above for why this can't be a runtime switch. -->
-      <xacro:if value="${'$(arg operating_mode)' == '2'}">
+           gripper_operating_mode arg's own comment above for why this can't be a runtime switch.
+           Note: when gripper_operating_mode=2, switch gripper_controller to
+           effort_controllers/JointGroupEffortController in control.yaml. -->
+      <xacro:if value="${'$(arg gripper_operating_mode)' == '2'}">
         <command_interface name="effort"/>
       </xacro:if>
-      <xacro:unless value="${'$(arg operating_mode)' == '2'}">
+      <xacro:unless value="${'$(arg gripper_operating_mode)' == '2'}">
         <command_interface name="position"/>
         <command_interface name="velocity"/>

Commit message: feat: e-stop target tracking, gripper GUI/joystick mode gating, PID tuning
- ik_teleop_node: while e-stopped, track the arm's live pose as target
  instead of the pre-e-stop target, so release holds in place instead
  of snapping back. Documented in README.
- gripper_teleop_node: gate joystick vs. GUI control on the arm's own
  joint_state_switch mode instead of racing on publish recency, fixing
  the joystick still winning briefly during GUI control.
- so100/so101: tuned servo PID (P=14, D=24) and deadband=10 for the
  position control loop.
- teleop.yaml: reduced max_target_reach to 0.45m.

File: so_arm_description/urdf/so100/so100.control.xacro (robot description, xacro)
@@ -26,5 +26,5 @@
   <xacro:property name="i_coefficient" value="0"/>
   <!-- Position insensitive-area (CW_DEAD/CCW_DEAD, both set to this value) -->
-  <xacro:property name="deadband" value="2"/>
+  <xacro:property name="deadband" value="10"/>
   <!-- Joint limits -->
   <xacro:property name="shoulder_pan_lower" value="-2"/>

File: so_arm_description/urdf/so101/so101.control.xacro (robot description, xacro)
@@ -26,5 +26,5 @@
   <xacro:property name="i_coefficient" value="0"/>
   <!-- Position insensitive-area (CW_DEAD/CCW_DEAD, both set to this value) -->
-  <xacro:property name="deadband" value="2"/>
+  <xacro:property name="deadband" value="10"/>
   <!-- Joint limits (from onshape-to-robot calibration) -->
   <xacro:property name="shoulder_pan_lower" value="-1.91986"/>
