Commit message: Move record/replay + add optional wrist camera to so_arm_bringup
record_replay_node, BagPlayer/BagRecorder, and their tests move from so_arm_control to
so_arm_bringup (ament_python) since they neither control nor calibrate the robot - so_arm_control
stays control-only. Adds opencv_camera_node, a cross-platform cv2.VideoCapture-based wrist camera
driver deployed via wrist_camera.launch.py, gated by two independent launch args: wrist_camera
(driver node, real hardware only - degrades to a clean exit + warning if no camera answers) and
wrist_camera_urdf (so101 only - strips the camera mount/links/joints from robot_description
entirely when false). CI, README, and package.xml updated to match.

File: so_arm_description/urdf/so100/so100.control.xacro (robot description, xacro)
@@ -15,8 +15,9 @@
   <xacro:property name="arm_operating_mode" value="0"/>     <!-- Arm joints 1-5: 0=Position, 1=Velocity, 2=PWM/Effort -->
   <xacro:property name="gripper_operating_mode" value="0"/> <!-- Gripper joint 6: 0=Position, 1=Velocity, 2=PWM/Effort -->
-  <!-- Motor-specific parameter (STS3215 default) -->
-  <xacro:property name="sts_max_velocity_steps" value="65535"/>  <!-- protocol's own u16 ceiling - let servo firmware, not us, set the real cap -->
+  <!-- Motor-specific, model-dependent parameter (written to every joint below so different
+       STS models could share this bus) -->
+  <xacro:property name="sts_protocol_max_vel_steps" value="65535"/>  <!-- protocol's own u16 ceiling - let servo firmware, not us, set the real cap -->
   <!-- Maximum allowable torque/velocity for each motor -->
-  <xacro:property name="max_velocity_steps" value="${sts_max_velocity_steps}"/>  <!-- full hardware max -->
+  <xacro:property name="max_velocity_steps" value="${sts_protocol_max_vel_steps}"/>  <!-- full hardware max -->
   <xacro:property name="max_velocity_rads" value="${max_velocity_steps*2*pi/4096}"/>  <!-- rad/s -->
   <xacro:property name="max_torque_nm" value="2.942"/>  <!-- N⋅m (30 kgf⋅cm for STS3215) -->

File: so_arm_description/urdf/so100/so100.urdf.xacro (robot description, xacro)
@@ -327,5 +327,4 @@
         <param name="use_sync_write">$(arg use_sync_write)</param>
         <param name="enable_mock_mode">$(arg use_mock)</param>
-        <param name="max_velocity_steps">${sts_max_velocity_steps}</param>
         <param name="reset_states_on_activate">true</param>
       </xacro:if>
@@ -336,4 +335,6 @@
       <param name="min_position">${shoulder_pan_lower}</param>
       <param name="max_position">${shoulder_pan_upper}</param>
+      <!-- Motor-specific, model-dependent parameter (per joint so different STS models can share this bus) -->
+      <param name="max_velocity_steps">${sts_protocol_max_vel_steps}</param>
       <param name="max_velocity">${max_velocity_rads}</param>
       <param name="position_center_steps">2048</param>
@@ -366,4 +367,6 @@
       <param name="min_position">${shoulder_lift_lower}</param>
       <param name="max_position">${shoulder_lift_upper}</param>
+      <!-- Motor-specific, model-dependent parameter (per joint so different STS models can share this bus) -->
+      <param name="max_velocity_steps">${sts_protocol_max_vel_steps}</param>
       <param name="max_velocity">${max_velocity_rads}</param>
       <param name="position_center_steps">2048</param>
@@ -396,4 +399,6 @@
       <param name="min_position">${elbow_flex_lower}</param>
       <param name="max_position">${elbow_flex_upper}</param>
+      <!-- Motor-specific, model-dependent parameter (per joint so different STS models can share this bus) -->
+      <param name="max_velocity_steps">${sts_protocol_max_vel_steps}</param>
       <param name="max_velocity">${max_velocity_rads}</param>
       <param name="position_center_steps">2048</param>
@@ -426,4 +431,6 @@
       <param name="min_position">${wrist_flex_lower}</param>
       <param name="max_position">${wrist_flex_upper}</param>
+      <!-- Motor-specific, model-dependent parameter (per joint so different STS models can share this bus) -->
+      <param name="max_velocity_steps">${sts_protocol_max_vel_steps}</param>
       <param name="max_velocity">${max_velocity_rads}</param>
       <param name="position_center_steps">2048</param>
@@ -456,4 +463,6 @@
       <param name="min_position">${wrist_roll_lower}</param>
       <param name="max_position">${wrist_roll_upper}</param>
+      <!-- Motor-specific, model-dependent parameter (per joint so different STS models can share this bus) -->
+      <param name="max_velocity_steps">${sts_protocol_max_vel_steps}</param>
       <param name="max_velocity">${max_velocity_rads}</param>
       <param name="position_center_steps">2048</param>
@@ -486,4 +495,6 @@
       <param name="min_position">${gripper_lower}</param>
       <param name="max_position">${gripper_upper}</param>
+      <!-- Motor-specific, model-dependent parameter (per joint so different STS models can share this bus) -->
+      <param name="max_velocity_steps">${sts_protocol_max_vel_steps}</param>
       <param name="max_velocity">${max_velocity_rads}</param>
       <param name="position_center_steps">2048</param>

File: so_arm_description/urdf/so101/so101.control.xacro (robot description, xacro)
@@ -15,8 +15,9 @@
   <xacro:property name="arm_operating_mode" value="0"/>     <!-- Arm joints 1-5: 0=Position, 1=Velocity, 2=PWM/Effort -->
   <xacro:property name="gripper_operating_mode" value="0"/> <!-- Gripper joint 6: 0=Position, 1=Velocity, 2=PWM/Effort -->
-  <!-- Motor-specific parameter (STS3215 default) -->
-  <xacro:property name="sts_max_velocity_steps" value="65535"/>  <!-- protocol's own u16 ceiling - let servo firmware, not us, set the real cap -->
+  <!-- Motor-specific, model-dependent parameter (written to every joint below so different
+       STS models could share this bus) -->
+  <xacro:property name="sts_protocol_max_vel_steps" value="65535"/>  <!-- protocol's own u16 ceiling - let servo firmware, not us, set the real cap -->
   <!-- Maximum allowable torque/velocity for each motor -->
-  <xacro:property name="max_velocity_steps" value="${sts_max_velocity_steps}"/>  <!-- full hardware max -->
+  <xacro:property name="max_velocity_steps" value="${sts_protocol_max_vel_steps}"/>  <!-- full hardware max -->
   <xacro:property name="max_velocity_rads" value="${max_velocity_steps*2*pi/4096}"/>  <!-- rad/s -->
   <xacro:property name="max_torque_nm" value="2.942"/>  <!-- N⋅m (30 kgf⋅cm for STS3215) -->

File: so_arm_description/urdf/so101/so101.urdf.xacro (robot description, xacro)
@@ -14,4 +14,6 @@
   <xacro:arg name="mujoco_model" default=""/>
   <xacro:arg name="mujoco_headless" default="false"/>
+  <!-- false = omit the wrist camera mount/body/frame links and their fixed joints below -->
+  <xacro:arg name="wrist_camera_urdf" default="true"/>
   <material name="light_grey">
     <color rgba="${light_grey_rgba}"/>
@@ -293,60 +295,62 @@
   </link>
   <!-- SO-101 wrist camera mount (Hex-Nut Recess, 32x32 UVC module form factor). -->
-  <link name="wrist_camera_mount_link">
-    <inertial>
-      <origin xyz="0 0 0" rpy="0 0 0"/>
-      <mass value="0.02"/>
-      <inertia ixx="1e-5" ixy="0" ixz="0" iyy="1e-5" iyz="0" izz="1e-5"/>
-    </inertial>
-    <visual>
-      <origin xyz="0 0 0" rpy="0 0 0"/>
-      <geometry>
-        <mesh filename="package://so_arm_description/meshes/so101/wrist_camera_mount_so101_v1.stl" scale="0.001 0.001 0.001"/>
-      </geometry>
-      <material name="light_grey"/>
-    </visual>
-    <collision>
-      <origin xyz="0 0 0" rpy="0 0 0"/>
-      <geometry>
-        <mesh filename="package://so_arm_description/meshes/so101/wrist_camera_mount_so101_v1.stl" scale="0.001 0.001 0.001"/>
-      </geometry>
-    </collision>
-  </link>
-  <link name="wrist_camera_body_link">
-    <inertial>
-      <origin xyz="0 0 0" rpy="0 0 0"/>
-      <mass value="0.015"/>
-      <inertia ixx="1e-5" ixy="0" ixz="0" iyy="1e-5" iyz="0" izz="1e-5"/>
-    </inertial>
-    <visual>
-      <origin xyz="0 0 0" rpy="0 0 0"/>
-      <geometry>
-        <mesh filename="package://so_arm_description/meshes/so101/wrist_camera_so101_v1.stl"/>
-      </geometry>
-      <material name="charcoal"/>
-    </visual>
-    <collision>
-      <origin xyz="0 0 0" rpy="0 0 0"/>
-      <geometry>
-        <mesh filename="package://so_arm_description/meshes/so101/wrist_camera_so101_v1.stl"/>
-      </geometry>
-    </collision>
-  </link>
-  <!-- Upstream-aligned wrist camera frame (+X forward, -Y right, +Z up). -->
-  <link name="wrist_camera_frame">
-    <inertial>
-      <origin xyz="0 0 0" rpy="0 0 0"/>
-      <mass value="1e-9"/>
-      <inertia ixx="0" ixy="0" ixz="0" iyy="0" iyz="0" izz="0"/>
-    </inertial>
-  </link>
-  <!-- REP-103 optical frame (+Z forward, +X right, +Y down). -->
-  <link name="wrist_camera_optical_frame">
-    <inertial>
-      <origin xyz="0 0 0" rpy="0 0 0"/>
-      <mass value="1e-9"/>
-      <inertia ixx="0" ixy="0" ixz="0" iyy="0" iyz="0" izz="0"/>
-    </inertial>
-  </link>
+  <xacro:if value="${'$(arg wrist_camera_urdf)' == 'true'}">
+    <link name="wrist_camera_mount_link">
+      <inertial>
+        <origin xyz="0 0 0" rpy="0 0 0"/>
+        <mass value="0.02"/>
+        <inertia ixx="1e-5" ixy="0" ixz="0" iyy="1e-5" iyz="0" izz="1e-5"/>
+      </inertial>
+      <visual>
+        <origin xyz="0 0 0" rpy="0 0 0"/>
+        <geometry>
+          <mesh filename="package://so_arm_description/meshes/so101/wrist_camera_mount_so101_v1.stl" scale="0.001 0.001 0.001"/>
+        </geometry>
+        <material name="light_grey"/>
+      </visual>
+      <collision>
+        <origin xyz="0 0 0" rpy="0 0 0"/>
+        <geometry>
+          <mesh filename="package://so_arm_description/meshes/so101/wrist_camera_mount_so101_v1.stl" scale="0.001 0.001 0.001"/>
+        </geometry>
+      </collision>
+    </link>
+    <link name="wrist_camera_body_link">
+      <inertial>
+        <origin xyz="0 0 0" rpy="0 0 0"/>
+        <mass value="0.015"/>
+        <inertia ixx="1e-5" ixy="0" ixz="0" iyy="1e-5" iyz="0" izz="1e-5"/>
+      </inertial>
+      <visual>
+        <origin xyz="0 0 0" rpy="0 0 0"/>
+        <geometry>
+          <mesh filename="package://so_arm_description/meshes/so101/wrist_camera_so101_v1.stl"/>
+        </geometry>
+        <material name="charcoal"/>
+      </visual>
+      <collision>
+        <origin xyz="0 0 0" rpy="0 0 0"/>
+        <geometry>
+          <mesh filename="package://so_arm_description/meshes/so101/wrist_camera_so101_v1.stl"/>
+        </geometry>
+      </collision>
+    </link>
+    <!-- Upstream-aligned wrist camera frame (+X forward, -Y right, +Z up). -->
+    <link name="wrist_camera_frame">
+      <inertial>
+        <origin xyz="0 0 0" rpy="0 0 0"/>
+        <mass value="1e-9"/>
+        <inertia ixx="0" ixy="0" ixz="0" iyy="0" iyz="0" izz="0"/>
+      </inertial>
+    </link>
+    <!-- REP-103 optical frame (+Z forward, +X right, +Y down). -->
+    <link name="wrist_camera_optical_frame">
+      <inertial>
+        <origin xyz="0 0 0" rpy="0 0 0"/>
+        <mass value="1e-9"/>
+        <inertia ixx="0" ixy="0" ixz="0" iyy="0" iyz="0" izz="0"/>
+      </inertial>
+    </link>
+  </xacro:if>
   <!-- Moving jaw link -->
   <link name="moving_jaw_link">
@@ -413,24 +417,26 @@
     <origin xyz="${end_effector_xyz}" rpy="${end_effector_rpy}"/>
   </joint>
-  <joint name="wrist_camera_mount_joint" type="fixed">
-    <parent link="gripper_link"/>
-    <child link="wrist_camera_mount_link"/>
-    <origin xyz="${wrist_camera_mount_xyz}" rpy="${wrist_camera_mount_rpy}"/>
-  </joint>
-  <joint name="wrist_camera_body_joint" type="fixed">
-    <parent link="wrist_camera_mount_link"/>
-    <child link="wrist_camera_body_link"/>
-    <origin xyz="${wrist_camera_body_xyz}" rpy="${wrist_camera_body_rpy}"/>
-  </joint>
-  <joint name="wrist_camera_frame_joint" type="fixed">
-    <parent link="gripper_link"/>
-    <child link="wrist_camera_frame"/>
-    <origin xyz="${wrist_camera_frame_xyz}" rpy="${wrist_camera_frame_rpy}"/>
-  </joint>
-  <joint name="wrist_camera_optical_joint" type="fixed">
-    <parent link="wrist_camera_frame"/>
-    <child link="wrist_camera_optical_frame"/>
-    <origin xyz="0 0 0" rpy="${wrist_camera_optical_rpy}"/>
-  </joint>
+  <xacro:if value="${'$(arg wrist_camera_urdf)' == 'true'}">
+    <joint name="wrist_camera_mount_joint" type="fixed">
+      <parent link="gripper_link"/>
+      <child link="wrist_camera_mount_link"/>
+      <origin xyz="${wrist_camera_mount_xyz}" rpy="${wrist_camera_mount_rpy}"/>
+    </joint>
+    <joint name="wrist_camera_body_joint" type="fixed">
+      <parent link="wrist_camera_mount_link"/>
+      <child link="wrist_camera_body_link"/>
+      <origin xyz="${wrist_camera_body_xyz}" rpy="${wrist_camera_body_rpy}"/>
+    </joint>
+    <joint name="wrist_camera_frame_joint" type="fixed">
+      <parent link="gripper_link"/>
+      <child link="wrist_camera_frame"/>
+      <origin xyz="${wrist_camera_frame_xyz}" rpy="${wrist_camera_frame_rpy}"/>
+    </joint>
+    <joint name="wrist_camera_optical_joint" type="fixed">
+      <parent link="wrist_camera_frame"/>
+      <child link="wrist_camera_optical_frame"/>
+      <origin xyz="0 0 0" rpy="${wrist_camera_optical_rpy}"/>
+    </joint>
+  </xacro:if>
   <joint name="gripper_joint" type="revolute">
     <parent link="gripper_link"/>
@@ -458,5 +464,4 @@
         <param name="use_sync_write">$(arg use_sync_write)</param>
         <param name="enable_mock_mode">$(arg use_mock)</param>
-        <param name="max_velocity_steps">${sts_max_velocity_steps}</param>
         <param name="reset_states_on_activate">true</param>
       </xacro:if>
@@ -467,4 +472,6 @@
       <param name="min_position">${shoulder_pan_lower}</param>
       <param name="max_position">${shoulder_pan_upper}</param>
+      <!-- Motor-specific, model-dependent parameter (per joint so different STS models can share this bus) -->
+      <param name="max_velocity_steps">${sts_protocol_max_vel_steps}</param>
       <param name="max_velocity">${max_velocity_rads}</param>
       <param name="position_center_steps">2048</param>
@@ -497,4 +504,6 @@
       <param name="min_position">${shoulder_lift_lower}</param>
       <param name="max_position">${shoulder_lift_upper}</param>
+      <!-- Motor-specific, model-dependent parameter (per joint so different STS models can share this bus) -->
+      <param name="max_velocity_steps">${sts_protocol_max_vel_steps}</param>
       <param name="max_velocity">${max_velocity_rads}</param>
       <param name="position_center_steps">2048</param>
@@ -527,4 +536,6 @@
       <param name="min_position">${elbow_flex_lower}</param>
       <param name="max_position">${elbow_flex_upper}</param>
+      <!-- Motor-specific, model-dependent parameter (per joint so different STS models can share this bus) -->
+      <param name="max_velocity_steps">${sts_protocol_max_vel_steps}</param>
       <param name="max_velocity">${max_velocity_rads}</param>
       <param name="position_center_steps">2048</param>
@@ -557,4 +568,6 @@
       <param name="min_position">${wrist_flex_lower}</param>
       <param name="max_position">${wrist_flex_upper}</param>
+      <!-- Motor-specific, model-dependent parameter (per joint so different STS models can share this bus) -->
+      <param name="max_velocity_steps">${sts_protocol_max_vel_steps}</param>
       <param name="max_velocity">${max_velocity_rads}</param>
       <param name="position_center_steps">2048</param>
@@ -587,4 +600,6 @@
       <param name="min_position">${wrist_roll_lower}</param>
       <param name="max_position">${wrist_roll_upper}</param>
+      <!-- Motor-specific, model-dependent parameter (per joint so different STS models can share this bus) -->
+      <param name="max_velocity_steps">${sts_protocol_max_vel_steps}</param>
       <param name="max_velocity">${max_velocity_rads}</param>
       <param name="position_center_steps">2048</param>
@@ -617,4 +632,6 @@
       <param name="min_position">${gripper_lower}</param>
       <param name="max_position">${gripper_upper}</param>
+      <!-- Motor-specific, model-dependent parameter (per joint so different STS models can share this bus) -->
+      <param name="max_velocity_steps">${sts_protocol_max_vel_steps}</param>
       <param name="max_velocity">${max_velocity_rads}</param>
       <param name="position_center_steps">2048</param>
