Commit message: Integrate wrist camera updates and tighten control safety

File: so_arm_description/mjcf/so_arm.mjcf.xacro (robot description, xacro)
@@ -130,4 +130,6 @@
       <mesh name="wrist_roll_pitch_so101_v2" file="$(find so_arm_description)/meshes/so101/wrist_roll_pitch_so101_v2.stl"/>
       <mesh name="wrist_roll_follower_so101_v1" file="$(find so_arm_description)/meshes/so101/wrist_roll_follower_so101_v1.stl"/>
+      <mesh name="wrist_camera_mount_so101_v1" file="$(find so_arm_description)/meshes/so101/wrist_camera_mount_so101_v1.stl"/>
+      <mesh name="wrist_camera_so101_v1" file="$(find so_arm_description)/meshes/so101/wrist_camera_so101_v1.stl"/>
       <mesh name="moving_jaw_so101_v1" file="$(find so_arm_description)/meshes/so101/moving_jaw_so101_v1.stl"/>
     </asset>
@@ -216,4 +218,18 @@
                   <geom class="collision" pos="0 -0.000218214 0.000949706" quat="0 1 0 0"
                         mesh="wrist_roll_follower_so101_v1" material="light_grey"/>
+                  <body name="wrist_camera_mount_link" pos="-0.0150 0.0240 -0.0315" quat="0.499798 -0.5002 0.499802 -0.5002">
+                    <inertial pos="0 0 0" mass="0.02" diaginertia="1e-5 1e-5 1e-5"/>
+                    <geom class="visual" pos="0 0 0" quat="1 0 0 0"
+                      mesh="wrist_camera_mount_so101_v1" material="light_grey"/>
+                    <geom class="collision" pos="0 0 0" quat="1 0 0 0"
+                      mesh="wrist_camera_mount_so101_v1" material="light_grey"/>
+                    <body name="wrist_camera_body_link" pos="-0.04941 -0.03813 0.0175" quat="0.379787 -0.596458 -0.379788 -0.596456">
+                      <inertial pos="0 0 0" mass="0.015" diaginertia="1e-5 1e-5 1e-5"/>
+                      <geom class="visual" pos="0 0 0" quat="1 0 0 0"
+                        mesh="wrist_camera_so101_v1" material="charcoal"/>
+                      <geom class="collision" pos="0 0 0" quat="1 0 0 0"
+                        mesh="wrist_camera_so101_v1" material="charcoal"/>
+                    </body>
+                  </body>
                   <!-- TCP marker, matches URDF's fixed end_effector_joint (end_effector_xyz/rpy
                        in so101.common.xacro) - not the ros2_so_arm MJCF's site, which does not
@@ -247,4 +263,7 @@
         <exclude body1="wrist_link" body2="gripper_link"/>
         <exclude body1="gripper_link" body2="moving_jaw_link"/>
+        <exclude body1="gripper_link" body2="wrist_camera_mount_link"/>
+        <exclude body1="wrist_camera_mount_link" body2="wrist_camera_body_link"/>
+        <exclude body1="gripper_link" body2="wrist_camera_body_link"/>
       </contact>
       <worldbody>

File: so_arm_description/urdf/so101/so101.common.xacro (robot description, xacro)
@@ -20,3 +20,15 @@
   <xacro:property name="end_effector_xyz" value="-0.0079 -0.000218121 -0.0981274"/>
   <xacro:property name="end_effector_rpy" value="0 1.5708 0"/>
+  <!-- SO-101 wrist camera (Hex-Nut Recess mount) reference pose from
+       TheRobotStudio SO-ARM100 + livekit-examples/so-frame. -->
+  <xacro:property name="wrist_camera_mount_xyz" value="-0.0150 0.0240 -0.0315"/>
+  <xacro:property name="wrist_camera_mount_rpy" value="-1.5708 -0.0008 -1.5708"/>
+  <!-- Camera body mesh pose and scale relative to wrist_camera_mount_link. -->
+     <xacro:property name="wrist_camera_body_xyz" value="-0.04941 -0.03813 0.0175"/>
+     <xacro:property name="wrist_camera_body_rpy" value="0 -1.5708 -2.0076"/>
+  <!-- Non-REP-103 camera frame that follows upstream so-frame alignment. -->
+  <xacro:property name="wrist_camera_frame_xyz" value="0.0025 0.0675 -0.0062"/>
+  <xacro:property name="wrist_camera_frame_rpy" value="3.141593 1.136305 -1.570797"/>
+  <!-- REP-103 optical frame (+Z forward, +X right, +Y down) as child of wrist_camera_frame. -->
+  <xacro:property name="wrist_camera_optical_rpy" value="-1.5708 0 -1.5708"/>
 </robot>

File: so_arm_description/urdf/so101/so101.urdf (robot description, URDF)
Before this commit: robot so101, 9 links, 8 joints
Links:
- added link wrist_camera_body_link, mass 0.015; collision mesh filename=../../meshes/so101/wrist_camera_so101_v1.stl; visual mesh filename=../../meshes/so101/wrist_camera_so101_v1.stl
- added link wrist_camera_frame, mass 1e-9
- added link wrist_camera_mount_link, mass 0.02; collision mesh filename=../../meshes/so101/wrist_camera_mount_so101_v1.stl scale=0.001 0.001 0.001; visual mesh filename=../../meshes/so101/wrist_camera_mount_so101_v1.stl scale=0.001 0.001 0.001
- added link wrist_camera_optical_frame, mass 1e-9
Joints:
- added joint wrist_camera_body_joint: type fixed, parent wrist_camera_mount_link, child wrist_camera_body_link, origin xyz=0 0 0 rpy=0 0 0
- added joint wrist_camera_frame_joint: type fixed, parent gripper_link, child wrist_camera_frame, origin xyz=0.0025 0.0675 -0.0062 rpy=3.141593 1.136305 -1.570797
- added joint wrist_camera_mount_joint: type fixed, parent gripper_link, child wrist_camera_mount_link, origin xyz=-0.0150 0.0240 -0.0315 rpy=-1.5708 -0.0008 -1.5708
- added joint wrist_camera_optical_joint: type fixed, parent wrist_camera_frame, child wrist_camera_optical_frame, origin xyz=0 0 0 rpy=-1.5708 0 -1.5708

File: so_arm_description/urdf/so101/so101.urdf.xacro (robot description, xacro)
@@ -300,4 +300,61 @@
     </inertial>
   </link>
+  <!-- SO-101 wrist camera mount (Hex-Nut Recess, 32x32 UVC module form factor). -->
+  <link name="wrist_camera_mount_link">
+    <inertial>
+      <origin xyz="0 0 0" rpy="0 0 0"/>
+      <mass value="0.02"/>
+      <inertia ixx="1e-5" ixy="0" ixz="0" iyy="1e-5" iyz="0" izz="1e-5"/>
+    </inertial>
+    <visual>
+      <origin xyz="0 0 0" rpy="0 0 0"/>
+      <geometry>
+        <mesh filename="package://so_arm_description/meshes/so101/wrist_camera_mount_so101_v1.stl" scale="0.001 0.001 0.001"/>
+      </geometry>
+      <material name="light_grey"/>
+    </visual>
+    <collision>
+      <origin xyz="0 0 0" rpy="0 0 0"/>
+      <geometry>
+        <mesh filename="package://so_arm_description/meshes/so101/wrist_camera_mount_so101_v1.stl" scale="0.001 0.001 0.001"/>
+      </geometry>
+    </collision>
+  </link>
+  <link name="wrist_camera_body_link">
+    <inertial>
+      <origin xyz="0 0 0" rpy="0 0 0"/>
+      <mass value="0.015"/>
+      <inertia ixx="1e-5" ixy="0" ixz="0" iyy="1e-5" iyz="0" izz="1e-5"/>
+    </inertial>
+    <visual>
+      <origin xyz="0 0 0" rpy="0 0 0"/>
+      <geometry>
+        <mesh filename="package://so_arm_description/meshes/so101/wrist_camera_so101_v1.stl"/>
+      </geometry>
+      <material name="charcoal"/>
+    </visual>
+    <collision>
+      <origin xyz="0 0 0" rpy="0 0 0"/>
+      <geometry>
+        <mesh filename="package://so_arm_description/meshes/so101/wrist_camera_so101_v1.stl"/>
+      </geometry>
+    </collision>
+  </link>
+  <!-- Upstream-aligned wrist camera frame (+X forward, -Y right, +Z up). -->
+  <link name="wrist_camera_frame">
+    <inertial>
+      <origin xyz="0 0 0" rpy="0 0 0"/>
+      <mass value="1e-9"/>
+      <inertia ixx="0" ixy="0" ixz="0" iyy="0" iyz="0" izz="0"/>
+    </inertial>
+  </link>
+  <!-- REP-103 optical frame (+Z forward, +X right, +Y down). -->
+  <link name="wrist_camera_optical_frame">
+    <inertial>
+      <origin xyz="0 0 0" rpy="0 0 0"/>
+      <mass value="1e-9"/>
+      <inertia ixx="0" ixy="0" ixz="0" iyy="0" iyz="0" izz="0"/>
+    </inertial>
+  </link>
   <!-- Moving jaw link -->
   <link name="moving_jaw_link">
@@ -363,4 +420,24 @@
     <child link="end_effector_link"/>
     <origin xyz="${end_effector_xyz}" rpy="${end_effector_rpy}"/>
+  </joint>
+  <joint name="wrist_camera_mount_joint" type="fixed">
+    <parent link="gripper_link"/>
+    <child link="wrist_camera_mount_link"/>
+    <origin xyz="${wrist_camera_mount_xyz}" rpy="${wrist_camera_mount_rpy}"/>
+  </joint>
+  <joint name="wrist_camera_body_joint" type="fixed">
+    <parent link="wrist_camera_mount_link"/>
+    <child link="wrist_camera_body_link"/>
+    <origin xyz="${wrist_camera_body_xyz}" rpy="${wrist_camera_body_rpy}"/>
+  </joint>
+  <joint name="wrist_camera_frame_joint" type="fixed">
+    <parent link="gripper_link"/>
+    <child link="wrist_camera_frame"/>
+    <origin xyz="${wrist_camera_frame_xyz}" rpy="${wrist_camera_frame_rpy}"/>
+  </joint>
+  <joint name="wrist_camera_optical_joint" type="fixed">
+    <parent link="wrist_camera_frame"/>
+    <child link="wrist_camera_optical_frame"/>
+    <origin xyz="0 0 0" rpy="${wrist_camera_optical_rpy}"/>
   </joint>
   <joint name="gripper_joint" type="revolute">
