Commit message: fix: invert axis for so101 joints 2-6 (shoulder_lift → gripper)
Motor 1 (shoulder_pan) direction matches visualization; motors 2-6 were
all physically opposite to the URDF. Negate axis xyz from '0 0 1' to
'0 0 -1' for:
  - shoulder_lift_joint
  - elbow_flex_joint
  - wrist_flex_joint
  - wrist_roll_joint
  - gripper_joint

Limits are symmetric around 0 on so101 so no limit swap is needed.

File: so_arm_description/urdf/so101/so101.urdf.xacro (robot description, xacro)
@@ -384,5 +384,5 @@
     <child link="upper_arm_link"/>
     <origin xyz="${shoulder_lift_xyz}" rpy="${shoulder_lift_rpy}"/>
-    <axis xyz="0 0 1"/>
+    <axis xyz="0 0 -1"/>
     <limit lower="${shoulder_lift_lower}" upper="${shoulder_lift_upper}" effort="${max_torque_nm}" velocity="1e6"/>
   </joint>
@@ -391,5 +391,5 @@
     <child link="lower_arm_link"/>
     <origin xyz="${elbow_flex_xyz}" rpy="${elbow_flex_rpy}"/>
-    <axis xyz="0 0 1"/>
+    <axis xyz="0 0 -1"/>
     <limit lower="${elbow_flex_lower}" upper="${elbow_flex_upper}" effort="${max_torque_nm}" velocity="1e6"/>
   </joint>
@@ -398,5 +398,5 @@
     <child link="wrist_link"/>
     <origin xyz="${wrist_flex_xyz}" rpy="${wrist_flex_rpy}"/>
-    <axis xyz="0 0 1"/>
+    <axis xyz="0 0 -1"/>
     <limit lower="${wrist_flex_lower}" upper="${wrist_flex_upper}" effort="${max_torque_nm}" velocity="1e6"/>
   </joint>
@@ -405,5 +405,5 @@
     <child link="gripper_link"/>
     <origin xyz="${wrist_roll_xyz}" rpy="${wrist_roll_rpy}"/>
-    <axis xyz="0 0 1"/>
+    <axis xyz="0 0 -1"/>
     <limit lower="${wrist_roll_lower}" upper="${wrist_roll_upper}" effort="${max_torque_nm}" velocity="1e6"/>
   </joint>
@@ -437,5 +437,5 @@
     <child link="moving_jaw_link"/>
     <origin xyz="${gripper_xyz}" rpy="${gripper_rpy}"/>
-    <axis xyz="0 0 1"/>
+    <axis xyz="0 0 -1"/>
     <limit lower="${gripper_lower}" upper="${gripper_upper}" effort="${max_torque_nm}" velocity="1e6"/>
   </joint>

Commit message: fix: revert gripper_joint axis inversion (0 0 -1 -> 0 0 1)

File: so_arm_description/urdf/so101/so101.urdf.xacro (robot description, xacro)
@@ -437,5 +437,5 @@
     <child link="moving_jaw_link"/>
     <origin xyz="${gripper_xyz}" rpy="${gripper_rpy}"/>
-    <axis xyz="0 0 -1"/>
+    <axis xyz="0 0 1"/>
     <limit lower="${gripper_lower}" upper="${gripper_upper}" effort="${max_torque_nm}" velocity="1e6"/>
   </joint>
