Commit message: chore: regenerate so101.urdf from current xacro (relative mesh paths)

File: so_arm_description/urdf/so101/so101.urdf (robot description, URDF)
Before this commit: robot so101, 13 links, 12 joints
Joints:
- joint elbow_flex_joint: axis 0 0 1 -> 0 0 -1
- joint gripper_joint: axis 0 0 1 -> 0 0 -1
- joint shoulder_lift_joint: axis 0 0 1 -> 0 0 -1
- joint wrist_camera_body_joint: origin xyz=0 0 0 rpy=0 0 0 -> xyz=-0.04941 -0.03813 0.0175 rpy=0 -1.5708 -2.0076
- joint wrist_flex_joint: axis 0 0 1 -> 0 0 -1
- joint wrist_roll_joint: axis 0 0 1 -> 0 0 -1
