Commit message: fix: invert gripper_joint limits to match negated axis (so101)
After negating gripper_joint axis to '0 0 -1', the physical limits
must be swapped and negated:
  lower: -0.174533 → -1.74533
  upper:  1.74533  →  0.174533

File: so_arm_description/urdf/so101/so101.control.xacro (robot description, xacro)
@@ -32,5 +32,5 @@
   <xacro:property name="wrist_roll_lower" value="-2.74385"/>
   <xacro:property name="wrist_roll_upper" value="2.84121"/>
-  <xacro:property name="gripper_lower" value="-0.174533"/>
-  <xacro:property name="gripper_upper" value="1.74533"/>
+  <xacro:property name="gripper_lower" value="-1.74533"/>
+  <xacro:property name="gripper_upper" value="0.174533"/>
 </robot>

File: so_arm_description/urdf/so101/so101.urdf (robot description, URDF)
Before this commit: robot so101, 13 links, 12 joints
Joints:
- joint gripper_joint: limit lower=-0.174533 upper=1.74533 effort=2.942 velocity=1e6 -> lower=-1.74533 upper=0.174533 effort=2.942 velocity=1e6
