Commit message: Fix so101 joint sign convention and harden so_arm_mujoco against model drift
so101's MJCF put every joint on axis="0 0 1", sign-flipping sim joint values
against so101.urdf and so against the real servos via sts_hardware_interface,
which nothing in so_arm_control compensated for (so100 was never affected). All
six joints are now axis="0 0 -1", and gripper_joint's range is back to the URDF's
-1.74533 0.174533.

That is deliberately not a copy of the URDF's axis attributes: shoulder_link's
body frame is turned 180 degrees from the URDF link frame, so reproducing the
same world rotation axis needs the opposite sign written here. Teleop keeps its
on-screen directions by compensating in teleop_ik.py rather than in the model,
and the gripper now closes toward its upper limit, matching so_arm_control's
_compute_gripper_target on the real arm.

Model/tooling:
- Fix wrist_cam pose, derived from the URDF's wrist_camera_optical_frame instead
  of guessed: it pointed back through the mount and sat 30mm off the lens.
- Reduce the drawn camera frustum (visual/scale/frustum), leaving fovy alone.
- Hide reference-frame sites (rgba alpha 0) so they stop rendering as spheres.
- Flatten mjcf/<model>/<model>.xml to mjcf/<model>.xml.
- Add `cli build --commit` to regenerate every committed model in one command;
  the committed files previously needed a manual build/sed/header dance and had
  silently drifted from the xacro.

Viewer:
- Extract HeldKeys/EStop into keyboard.py, shared by preview and teleop.
- Add an e-stop to the plain preview, and an M-key mode toggle in teleop that
  hands the joints to the viewer's own Control sidebar.
- Stop rewriting data.ctrl every frame, so those sliders actually take effect.
- Keep the e-stop releasing torque (arm falls) rather than holding position:
  that models cutting power to the STS3215s, unlike pt_mujoco's pan-tilt.
- Fix two e-stop defects: dof_frictionloss was zeroed alongside dof_damping,
  leaving an undamped arm swinging for seconds, and releasing after a long fall
  snapped the arm toward a stale tracker target (44 rad/s spike).

Tests (60, up from 8):
- test_generated_assets.py fails if a committed model drifts from the xacro.
- test_urdf_agreement.py reimplements the URDF kinematics and checks link poses,
  joint axes, limits, full FK, the camera optical frame and the end-effector site.
- Cover keyboard/e-stop, benchmark_mujoco and the invisible-site regression.

Add benchmark_mujoco.py for per-joint step-response measurement.

File: so_arm_mujoco/mjcf/so_arm.mjcf.xacro (robot description, xacro)
@@ -10,5 +10,9 @@
   <xacro:property name="so_arm_config" value="$(arg so_arm_config)"/>
   <compiler angle="radian"/>
-  <option cone="elliptic" impratio="10"/>
+  <!-- implicitfast trades a bit of speed for much better stability on stiff position actuators
+       like the STS3215 servos below - Euler (MuJoCo's default) needs a much smaller timestep to
+       stay stable at these gains, which is what drove the steady-state tracking error fights in
+       teleop_ik.py before this was pinned down explicitly. -->
+  <option timestep="0.002" integrator="implicitfast" iterations="60" cone="elliptic" impratio="10"/>
   <asset>
     <material name="light_grey" rgba="0.8 0.8 0.8 1.0"/>
@@ -86,5 +90,10 @@
                   <geom mesh="Fixed_Jaw_Motor" material="charcoal" class="visual" quat="0.707107 0.707107 0 0"/>
                   <!-- TCP marker, matches URDF's end_effector_joint; estimated, not calibrated. -->
-                  <site group="5" name="end_effector_link" pos="0.0025 0.0 -0.106" quat="0.707107 0 0.707107 0"/>
+                  <!-- rgba alpha=0: this is a kinematic reference frame (CONNECT-constraint
+                       anchor, ee_pose()), not something meant to be looked at - invisible
+                       regardless of the viewer's own site-group visibility toggle, rather than
+                       relying on group=5 being off by the viewer's own (overridable) default. -->
+                  <site group="5" name="end_effector_link" pos="0.0025 0.0 -0.106"
+                        quat="0.707107 0 0.707107 0" rgba="0 0 0 0"/>
                   <body name="moving_jaw_link" pos="-0.0202 0 -0.0244" quat="0 0 0.707107 0.707107">
                     <joint name="gripper_joint" axis="0 0 1" range="-0.2 2.0" class="sts3215"/>
@@ -133,4 +142,18 @@
     </asset>
     <!-- Ported from ros2_so_arm's so_arm101.xml, verified against our URDF (gripper_joint recomputed below). -->
+    <!-- Every joint below is axis="0 0 -1", and must stay that way. They were all "0 0 1"
+         until a URDF cross-check caught it, which silently sign-flipped sim joint values
+         against so101.urdf - and so against the real servos through sts_hardware_interface,
+         which nothing in so_arm_control compensates for. so100 never had the problem.
+         Note this is NOT simply copying so101.urdf's axis attributes: the URDF gives
+         shoulder_pan "0 0 1" and the other five "0 0 -1". What has to match is the *world*
+         rotation axis, and some bodies here don't share the URDF link's frame (shoulder_link
+         is turned 180 degrees), so an axis written in this file's frame can need the opposite
+         sign to produce the same physical rotation. The rule, which test_urdf_agreement.py
+         enforces directly:
+             axis_mjcf = R_body_mjcf^T . (R_link_urdf . axis_urdf)
+         Re-deriving that for so101 gives "0 0 -1" six times over. Do not "tidy" these to match
+         the URDF text - that re-breaks sim-to-real. If a teleop direction needs reversing,
+         negate it in teleop_ik.py, where the compensation is visible and tested. -->
     <xacro:macro name="so_arm101_body">
       <body name="base_link">
@@ -146,5 +169,5 @@
               mesh="waveshare_mounting_plate_so101_v2" material="light_grey"/>
         <body name="shoulder_link" pos="0.0388353 -8.97657e-09 0.0624" quat="0 0 -1 0">
-          <joint axis="0 0 1" name="shoulder_pan_joint" range="-1.91986 1.91986" class="sts3215"/>
+          <joint axis="0 0 -1" name="shoulder_pan_joint" range="-1.91986 1.91986" class="sts3215"/>
           <inertial pos="-0.0307604 -1.66727e-05 -0.0252713" mass="0.100006"
                     fullinertia="8.3759e-05 8.10403e-05 2.39783e-05 7.55525e-08 -1.16342e-06 1.54663e-07"/>
@@ -162,5 +185,5 @@
                 mesh="rotation_pitch_so101_v1" material="light_grey"/>
           <body name="upper_arm_link" pos="-0.0303992 -0.0182778 -0.0542" quat="0.5 -0.5 -0.5 -0.5">
-            <joint axis="0 0 1" name="shoulder_lift_joint" range="-1.74533 1.74533" class="sts3215"/>
+            <joint axis="0 0 -1" name="shoulder_lift_joint" range="-1.74533 1.74533" class="sts3215"/>
             <inertial pos="-0.0898471 -0.00838224 0.0184089" mass="0.103"
                       fullinertia="4.08002e-05 0.000147318 0.000142487 -1.97819e-05 -4.03016e-08 8.97326e-09"/>
@@ -174,5 +197,5 @@
                   mesh="upper_arm_so101_v1" material="light_grey"/>
             <body name="lower_arm_link" pos="-0.11257 -0.028 0" quat="0.707107 0 0 0.707107">
-              <joint axis="0 0 1" name="elbow_flex_joint" range="-1.69 1.69" class="sts3215"/>
+              <joint axis="0 0 -1" name="elbow_flex_joint" range="-1.69 1.69" class="sts3215"/>
               <inertial pos="-0.0980701 0.00324376 0.0182831" mass="0.104"
                         fullinertia="2.87438e-05 0.000159844 0.00014529 7.41152e-06 1.26409e-06 -4.90188e-08"/>
@@ -190,5 +213,5 @@
                     mesh="sts3215_03a_v1" material="charcoal"/>
               <body name="wrist_link" pos="-0.1349 0.0052 0" quat="0.707388 0 0 -0.706825">
-                <joint axis="0 0 1" name="wrist_flex_joint" range="-1.65806 1.65806" class="sts3215"/>
+                <joint axis="0 0 -1" name="wrist_flex_joint" range="-1.65806 1.65806" class="sts3215"/>
                 <inertial pos="-0.000103312 -0.0386143 0.0281156" mass="0.079"
                           fullinertia="3.68263e-05 2.5391e-05 2.1e-05 1.7893e-08 -5.28128e-08 3.6412e-06"/>
@@ -203,5 +226,5 @@
                 <!-- quat carries so101_new_calib.xml's wrist_roll calibration offset (matches URDF). -->
                 <body name="gripper_link" pos="0 -0.0611 0.0181" quat="0.0172091 -0.0172091 0.706897 0.706897">
-                  <joint axis="0 0 1" name="wrist_roll_joint" range="-2.74385 2.84121" class="sts3215"/>
+                  <joint axis="0 0 -1" name="wrist_roll_joint" range="-2.74385 2.84121" class="sts3215"/>
                   <inertial pos="0.000213627 0.000245138 -0.025187" mass="0.087"
                             fullinertia="2.75087e-05 4.33657e-05 3.45059e-05 -3.35241e-07 -5.7352e-06 -5.17847e-08"/>
@@ -227,12 +250,39 @@
                         <geom class="collision" pos="0 0 0" quat="1 0 0 0"
                           mesh="wrist_camera_so101_v1" material="charcoal"/>
+                        <!-- Derived from the URDF's wrist_camera_optical_frame, not guessed.
+                             The URDF hangs wrist_camera_frame directly off gripper_link, while
+                             MuJoCo needs the camera nested under wrist_camera_body_link - so
+                             the URDF chain is rebased onto this body rather than copied:
+                               T_body_optical = inv(T_grip_mount . T_mount_body)
+                                                . T_grip_frame . T_frame_optical
+                             using so101.common.xacro's wrist_camera_{mount,body,frame}_* and
+                             wrist_camera_optical_rpy (URDF fixed-axis XYZ rpy). That chain
+                             reproduces this file's own mount/body quats to 6 decimals, which
+                             is what confirms the convention is right. Final term converts
+                             REP-103 optical (+Z fwd, +Y down) to MuJoCo's camera convention
+                             (-Z fwd, +Y up): a 180deg turn about the optical frame's own X,
+                             hence quat ~ (0,-1,0,0); the small w/z terms carry the -0.0008 rad
+                             yaw the real mount has. pos lands 14.1mm along this body's +Z -
+                             an earlier revision put it 30mm along +Y instead, which is what
+                             left the rendered frustum visibly offset from the lens mesh.
+                             fovy=86.67 derived from wrist_camera_calibration.yaml's fy=508.7 at
+                             960px height: 2*atan((960/2)/508.7). Resolution downscaled from the
+                             real 1280x960 capture - full-res offscreen rendering every sim step
+                             isn't worth the cost for a placeholder FOV/calibration. -->
+                        <camera name="wrist_cam" fovy="86.67" resolution="640 480"
+                                pos="0 -0.0000395 0.0141025"
+                                quat="0.00155434 -0.99999879 0 0.00000597"/>
                       </body>
                     </body>
                   </xacro:if>
-                  <!-- Matches URDF's end_effector_joint rpy, unlike ros2_so_arm's MJCF site. -->
-                  <site group="5" name="end_effector_link" pos="-0.0079 -0.000218121 -0.0981274" quat="0.707105 0 0.707108 0"/>
+                  <!-- Matches URDF's end_effector_joint rpy, unlike ros2_so_arm's MJCF site.
+                       rgba alpha=0: kinematic reference frame, not meant to be looked at - see
+                       the so100 branch's site above for why this is invisible outright rather
+                       than relying on the viewer's (overridable) group=5 default. -->
+                  <site group="5" name="end_effector_link" pos="-0.0079 -0.000218121 -0.0981274"
+                        quat="0.707105 0 0.707108 0" rgba="0 0 0 0"/>
                   <!-- Recomputed from our own gripper_rpy (no pitch offset), unlike ros2_so_arm's macro. -->
                   <body name="moving_jaw_link" pos="0.0202 0.0188 -0.0234" quat="0.707105 0.707108 0 0">
-                    <joint axis="0 0 1" name="gripper_joint" range="-0.174533 1.74533" class="sts3215"/>
+                    <joint axis="0 0 -1" name="gripper_joint" range="-1.74533 0.174533" class="sts3215"/>
                     <inertial pos="-0.00157495 -0.0300244 0.0192755" mass="0.012"
                               fullinertia="6.61427e-06 1.89032e-06 5.28738e-06 -3.19807e-07 -5.90717e-09 -1.09945e-07"/>
@@ -275,4 +325,10 @@
       <rgba haze="0.15 0.25 0.35 1"/>
       <global azimuth="45" elevation="-20"/>
+      <!-- How far the wrist_cam frustum is *drawn* when the viewer's Camera visualization is
+           on - purely cosmetic, unrelated to the camera's actual fovy/calibration or to what
+           it renders. MuJoCo's default (10) is well past saturation at this model's 0.5m
+           extent, so the frustum swamps the arm; 2 keeps it legible at roughly half the
+           on-screen footprint. Lower it further (1 is small but still visible) to taste. -->
+      <scale frustum="2"/>
     </visual>
     <asset>

Commit message: Add per-package READMEs and mujoco_ros2_control plugin parity with lekiwi/pantilt
Documentation:
- Add so_arm_description, so_arm_control and so_arm_bringup READMEs,
  matching lekiwi_ros2/pantilt_ros2's structure and style; update the
  top-level README and so_arm_mujoco's to match.
- Fact-checked every README against the actual source (launch args,
  config defaults, joystick mappings, test coverage) rather than
  trusting what was drafted; fixed three real inaccuracies this
  surfaced in so_arm_description's README (a --write regeneration
  command that doesn't exist, a Tests section claiming coverage that
  isn't there, and a wrong frame-nesting diagram for the wrist camera).

mujoco_ros2_control plugin parity:
- Add a simulated /emergency_stop (mujoco_ros2_plugins/EmergencyStopPlugin)
  to ros2_control_hardware_type:=mujoco, wired the same way lekiwi_ros2
  and pantilt_ros2 do. It holds the last commanded position rather than
  releasing torque - matching mujoco_ros2_plugins' behavior for their
  position-controlled joints, not this arm's actual gravity-drop on
  power cut - documented explicitly so it isn't mistaken for hardware
  validation.
- Add a simulated wrist camera (mujoco_ros2_control_plugins/CameraPlugin,
  SO101 + wrist_camera_urdf:=true only) on the same /image_raw and
  /camera_info topics the real driver uses.
- so_arm_control/package.xml gains mujoco_ros2_control_plugins and
  mujoco_ros2_plugins as exec_depends, matching pantilt_ros2's
  pt_control dependency set exactly.

mujoco_arena launch argument:
- New named MJCF scenes (mjcf/scenes/flat.mjcf.xacro, arena.mjcf.xacro),
  replacing the old boolean scene:=true/false toggle. arena is a small
  tabletop workspace - three graspable cubes and a tray - placed within
  SO101's measured reach (a joint-range sweep puts the end effector at
  radius 0.0-0.46m at tabletop height, matching teleop.yaml's own
  max_target_reach: 0.45), not lekiwi/pantilt's walled-room-with-obstacles
  arena, which is for mobile-base navigation-recovery testing and has no
  bearing on a stationary arm.
- Exposed as a boolean mujoco_arena launch argument (default false) in
  control.launch.py, so_arm.launch.py and leader_follower.launch.py
  (with leader_/follower_ prefixes, alongside the existing
  leader_/follower_mujoco_headless), translating internally to the
  richer flat/arena/none scene selector. The standalone so_arm_mujoco
  CLI (cli.py, teleop_ik.py) and Python API (build_model_xml,
  SoArmEnv/SoArmVecEnv) keep that full selector via --scene/scene=,
  matching lekiwi_mujoco/pt_mujoco's own convention - and stay entirely
  ROS-free, same as before.
- Regenerated the committed mjcf/so100.xml and mjcf/so101.xml for the
  new scene-composition mechanism.

Verified end-to-end, not just statically: rebuilt so_arm_control,
so_arm_bringup and so_arm_mujoco and confirmed via real
`ros2 launch --show-arguments` that mujoco_arena and mujoco_headless
are correctly declared at all three launch-file levels, and via the
real xacro/ament_index toolchain that scene=flat/arena/none all
compile to valid MuJoCo models. Fixed a real regression this caught:
test_leader_follower_launch.py's exact-set-equality assertion on
declared argument names, which the two new leader_/follower_mujoco_arena
args would otherwise have broken.

File: so_arm_mujoco/mjcf/so_arm.mjcf.xacro (robot description, xacro)
@@ -5,5 +5,7 @@
 <mujoco xmlns:xacro="http://www.ros.org/wiki/xacro" model="so_arm">
   <xacro:arg name="so_arm_config" default="so101"/>
-  <xacro:arg name="scene" default="true"/>
+  <!-- flat (skybox+floor, the default), arena (flat + graspable cubes/tray, see
+       mjcf/scenes/), or none (omit entirely, e.g. to compose into an external scene). -->
+  <xacro:arg name="scene" default="flat"/>
   <!-- so101 only; mirrors urdf's wrist_camera_urdf arg. False omits the camera bodies below. -->
   <xacro:arg name="wrist_camera_mjcf" default="true"/>
@@ -318,28 +320,11 @@
     </worldbody>
   </xacro:if>
-  <!-- Compares $(arg scene) directly - xacro auto-coerces bridged properties to Python bool. -->
-  <xacro:if value="${'$(arg scene)' == 'true'}">
-    <statistic center="0.1 -0.01 0.05" extent="0.5"/>
-    <visual>
-      <headlight diffuse="0.6 0.6 0.6" ambient="0.3 0.3 0.3" specular="0 0 0"/>
-      <rgba haze="0.15 0.25 0.35 1"/>
-      <global azimuth="45" elevation="-20"/>
-      <!-- How far the wrist_cam frustum is *drawn* when the viewer's Camera visualization is
-           on - purely cosmetic, unrelated to the camera's actual fovy/calibration or to what
-           it renders. MuJoCo's default (10) is well past saturation at this model's 0.5m
-           extent, so the frustum swamps the arm; 2 keeps it legible at roughly half the
-           on-screen footprint. Lower it further (1 is small but still visible) to taste. -->
-      <scale frustum="2"/>
-    </visual>
-    <asset>
-      <texture type="skybox" builtin="gradient" rgb1="0.3 0.5 0.7" rgb2="0 0 0" width="512" height="3072"/>
-      <texture type="2d" name="groundplane" builtin="checker" mark="edge" rgb1="0.2 0.3 0.4" rgb2="0.1 0.2 0.3"
-        markrgb="0.8 0.8 0.8" width="300" height="300"/>
-      <material name="groundplane" texture="groundplane" texuniform="true" texrepeat="5 5" reflectance="0.2"/>
-    </asset>
-    <worldbody>
-      <light pos="0 0 1.5" dir="0 0 -1" directional="true"/>
-      <geom name="floor" size="0 0 0.05" type="plane" material="groundplane"/>
-    </worldbody>
+  <!-- Named scenes live in mjcf/scenes/ - see simulation.py's build_model_xml for how the
+       "scene" arg's value reaches here (it's resolved to a filename, not compared directly). -->
+  <xacro:if value="${'$(arg scene)' == 'flat'}">
+    <xacro:include filename="$(find so_arm_mujoco)/mjcf/scenes/flat.mjcf.xacro"/>
+  </xacro:if>
+  <xacro:if value="${'$(arg scene)' == 'arena'}">
+    <xacro:include filename="$(find so_arm_mujoco)/mjcf/scenes/arena.mjcf.xacro"/>
   </xacro:if>
 </mujoco>
